Commit message: update mover-controller

File: noid_description/urdf/typeC_lifter/virtual_lifter.urdf.xacro (robot description, xacro)
@@ -14,5 +14,5 @@
        xmlns:physics="http://playerstage.sourceforge.net/gazebo/xmlschema/#physics"
        xmlns:xacro="http://ros.org/wiki/xacro">
-  <xacro:include filename="$(find aero_description)/urdf/common.xacro" />
+  <xacro:include filename="$(find noid_description)/robots/common.xacro" />
   <xacro:macro name="virtual_lifter" params="base_link x_max x_min z_max z_min">
     <link name="${base_link}" />

File: noid_description/urdf/typeE_wheel/wheels.urdf.xacro (robot description, xacro)
@@ -14,9 +14,9 @@
        xmlns:physics="http://playerstage.sourceforge.net/gazebo/xmlschema/#physics"
        xmlns:xacro="http://ros.org/wiki/xacro">
-  <xacro:include filename="$(find aero_description)/urdf/common.xacro" />
-  <xacro:include filename="$(find aero_description)/common_urdf/gazebo.xacro" />
+  <xacro:include filename="$(find noid_description)/robots/common.xacro" />
+  <xacro:include filename="$(find noid_description)/urdf/gazebo.xacro" />
   <xacro:property name="wheel_radius" value="0.075"/>
   <xacro:macro name="wheels" params="base_link disable_mesh:=false">
-  <!-- ============================   aero(typeE_wheels)   ============================ -->
+  <!-- ============================   typeE_wheels  ============================ -->
   <link name="${base_link}"/>
     <link name="wheel_base_link">
@@ -24,5 +24,5 @@
         <origin xyz="0.0 0.0 0.0" rpy="0 -0 0"/>
         <geometry>
-          <mesh filename="package://aero_description/meshes/typeE_wheel/wheels_base.dae" scale="1 1 1" />
+          <mesh filename="package://noid_description/meshes/typeE_wheel/wheels_base.dae" scale="1 1 1" />
           </geometry>
       </visual> </xacro:unless>
@@ -30,5 +30,5 @@
         <!--origin xyz="0.0 0.0 0.0" rpy="0 -0 0"/>
         <geometry>
-          <mesh filename="package://aero_description/meshes/typeE_wheel/wheels_base.dae" scale="1 1 1" />
+          <mesh filename="package://noid_description/meshes/typeE_wheel/wheels_base.dae" scale="1 1 1" />
         </geometry-->
         <origin xyz="0.018 0.0 0.0375" rpy="0 -0 0"/>
@@ -48,5 +48,5 @@
         <origin xyz="0.0 0.0 0.0" rpy="0 -0 0"/>
         <geometry>
-          <mesh filename="package://aero_description/meshes/typeE_wheel/wheels_top.dae" scale="1 1 1" />
+          <mesh filename="package://noid_description/meshes/typeE_wheel/wheels_top.dae" scale="1 1 1" />
         </geometry>
       </visual> </xacro:unless>
@@ -63,5 +63,5 @@
         <origin xyz="0.0 0.0 0.0" rpy="-1.57079632679 0 0"/>
         <geometry>
-          <mesh filename="package://aero_description/meshes/typeE_wheel/wheels_mecanum.dae" scale="1 1 1" />
+          <mesh filename="package://noid_description/meshes/typeE_wheel/wheels_mecanum.dae" scale="1 1 1" />
         </geometry>
       </visual> </xacro:unless>
@@ -84,5 +84,5 @@
         <origin xyz="0.0 0.0 0.0" rpy="-1.57079632679 0 0"/>
         <geometry>
-          <mesh filename="package://aero_description/meshes/typeE_wheel/wheels_mecanum.dae" scale="1 1 1" />
+          <mesh filename="package://noid_description/meshes/typeE_wheel/wheels_mecanum.dae" scale="1 1 1" />
         </geometry>
       </visual> </xacro:unless>
@@ -105,5 +105,5 @@
         <origin xyz="0.0 0.0 0.0" rpy="-1.57079632679 0 0"/>
         <geometry>
-          <mesh filename="package://aero_description/meshes/typeE_wheel/wheels_mecanum.dae" scale="1 1 1" />
+          <mesh filename="package://noid_description/meshes/typeE_wheel/wheels_mecanum.dae" scale="1 1 1" />
         </geometry>
       </visual> </xacro:unless>
@@ -126,5 +126,5 @@
         <origin xyz="0.0 0.0 0.0" rpy="-1.57079632679 0 0"/>
         <geometry>
-          <mesh filename="package://aero_description/meshes/typeE_wheel/wheels_mecanum.dae" scale="1 1 1" />
+          <mesh filename="package://noid_description/meshes/typeE_wheel/wheels_mecanum.dae" scale="1 1 1" />
         </geometry>
       </visual> </xacro:unless>
@@ -147,5 +147,5 @@
         <origin xyz="0.0 0.0 0.0" rpy="0 0 0"/>
         <geometry>
-          <mesh filename="package://aero_description/meshes/typeE_wheel/wheels_urg.dae" scale="1 1 1" />
+          <mesh filename="package://noid_description/meshes/typeE_wheel/wheels_urg.dae" scale="1 1 1" />
         </geometry>
       </visual> </xacro:unless>
