Commit message: noid?hand_controller update

File: noid_description/robots/typeF/aero.urdf.xacro (robot description, xacro)
@@ -4,15 +4,15 @@
        xmlns:interface="http://playerstage.sourceforge.net/gazebo/xmlschema/#interface"
        xmlns:xacro="http://playerstage.sourceforge.net/gazebo/xmlschema/#interface"
-       name="AeroTypeFCET" >
+       name="SEED-Noid-typeFCET" >
   <!-- The following included files set up definitions of parts of the robot body -->
   <!-- common variables -->
   <xacro:include filename="$(find noid_description)/robots/typeF/common.xacro" />
   <!-- wraps upperbody and hand-->
-  <xacro:include filename="$(find noid_description)/robots/typeF/aero-upper.urdf.xacro" />
+  <xacro:include filename="$(find noid_description)/robots/typeF/noid-upper.urdf.xacro" />
   <!-- wraps lifter and wheels-->
-  <xacro:include filename="$(find noid_description)/robots/typeF/aero-wheels.urdf.xacro" />
+  <xacro:include filename="$(find noid_description)/robots/typeF/noid-wheels.urdf.xacro" />
  <!-- Now we can start using the macros included above to define the actual robot -->
- <xacro:aero-upper/>
- <xacro:aero-wheels base_link="base_link"/>
+ <xacro:noid-upper/>
+ <xacro:noid-wheels base_link="base_link"/>
  <!-- gazebo settings -->
  <!-- camera -->

File: noid_description/urdf/trx_s/trx_s.urdf.xacro (robot description, xacro)
@@ -5,6 +5,6 @@
        xmlns:interface="http://playerstage.sourceforge.net/gazebo/xmlschema/#interface"
        xmlns:xacro="http://ros.org/wiki/xacro">
-  <xacro:include filename="$(find aero_description)/urdf/common.xacro" />
-  <xacro:include filename="$(find aero_description)/common_urdf/gazebo.xacro" />
+  <xacro:include filename="$(find noid_description)/robots/typeF/common.xacro" />
+  <xacro:include filename="$(find noid_description)/urdf/gazebo.xacro" />
   <property name="M_PI" value="3.1415926535897931" />
   <xacro:macro name="trx_s" params="prefix:=r reflect:=1 disable_mesh:=false">
@@ -16,5 +16,5 @@
       <origin xyz="0 0 0" rpy="0 -0 ${(1.0 - reflect) * M_PI / 2.0}"/>
       <geometry>
-        <mesh filename="package://aero_description/meshes/trx_s/RARM_LINK7_mesh.dae" scale="1 1 1" />
+        <mesh filename="package://noid_description/meshes/trx_s/RARM_LINK7_mesh.dae" scale="1 1 1" />
       </geometry>
     </visual> </xacro:unless>
@@ -44,5 +44,5 @@
       <origin xyz="0 ${0.013 * reflect} 0.115" rpy="0 -0 ${(1.0 - reflect) * M_PI / 2.0}"/>
       <geometry>
-        <mesh filename="package://aero_description/meshes/trx_s/RARM_INDEX_LINK1_mesh.dae" scale="1 1 1" />
+        <mesh filename="package://noid_description/meshes/trx_s/RARM_INDEX_LINK1_mesh.dae" scale="1 1 1" />
       </geometry>
     </visual> </xacro:unless>
@@ -64,5 +64,5 @@
       <origin xyz="0 ${-0.015754 * reflect} 0.149615" rpy="0 -0 ${(1.0 - reflect) * M_PI / 2.0}"/>
       <geometry>
-        <mesh filename="package://aero_description/meshes/trx_s/RARM_INDEX_LINK2_mesh.dae" scale="1 1 1" />
+        <mesh filename="package://noid_description/meshes/trx_s/RARM_INDEX_LINK2_mesh.dae" scale="1 1 1" />
       </geometry>
     </visual> </xacro:unless>
@@ -84,5 +84,5 @@
       <origin xyz="0 ${-0.03747 * reflect} 0.162972" rpy="0 -0 ${(1.0 - reflect) * M_PI / 2.0}"/>
       <geometry>
-        <mesh filename="package://aero_description/meshes/trx_s/RARM_INDEX_LINK3_mesh.dae" scale="1 1 1" />
+        <mesh filename="package://noid_description/meshes/trx_s/RARM_INDEX_LINK3_mesh.dae" scale="1 1 1" />
       </geometry>
     </visual> </xacro:unless>
@@ -104,5 +104,5 @@
       <origin xyz="0 ${-0.022355 * reflect} 0.079645" rpy="0 -0 ${(1.0 - reflect) * M_PI / 2.0}"/>
       <geometry>
-        <mesh filename="package://aero_description/meshes/trx_s/RARM_THUMB_LINK_mesh.dae" scale="1 1 1" />
+        <mesh filename="package://noid_description/meshes/trx_s/RARM_THUMB_LINK_mesh.dae" scale="1 1 1" />
       </geometry>
     </visual> </xacro:unless>

File: noid_description/urdf/typeC_lifter/lifter.urdf.xacro (robot description, xacro)
@@ -14,19 +14,19 @@
        xmlns:physics="http://playerstage.sourceforge.net/gazebo/xmlschema/#physics"
        xmlns:xacro="http://ros.org/wiki/xacro">
-  <xacro:include filename="$(find aero_description)/urdf/common.xacro" />
-  <xacro:include filename="$(find aero_description)/common_urdf/gazebo.xacro" />
+  <xacro:include filename="$(find noid_description)/robots/typeF/common.xacro" />
+  <xacro:include filename="$(find noid_description)/urdf/gazebo.xacro" />
   <xacro:macro name="lifter" params="base_link">
-  <!-- ============================   aero(typeC_lifter)   ============================ -->
+  <!-- ============================   (typeC_lifter)   ============================ -->
     <link name="${base_link}">
       <visual>
         <origin xyz="0 0 0" rpy="0 -0 0"/>
         <geometry>
-          <mesh filename="package://aero_description/meshes/typeC_lifter/lifter_base.dae" scale="1 1 1" />
-        </geometry>
-      </visual>
-      <collision>
-        <origin xyz="0 0 0" rpy="0 -0 0"/>
-        <geometry>
-          <mesh filename="package://aero_description/meshes/typeC_lifter/lifter_base.dae" scale="1 1 1" />
+          <mesh filename="package://noid_description/meshes/typeC_lifter/lifter_base.dae" scale="1 1 1" />
+        </geometry>
+      </visual>
+      <collision>
+        <origin xyz="0 0 0" rpy="0 -0 0"/>
+        <geometry>
+          <mesh filename="package://noid_description/meshes/typeC_lifter/lifter_base.dae" scale="1 1 1" />
         </geometry>
       </collision>
@@ -42,11 +42,11 @@
         <origin xyz="0.0 0.0 0" rpy="3.1415 -0 0"/>
         <geometry>
-          <mesh filename="package://aero_description/meshes/typeC_lifter/lifter_bone.dae" scale="1 1 1" />
-        </geometry>
-      </visual>
-      <collision>
-        <origin xyz="0.0 0.0 0" rpy="3.1415 -0 0"/>
-        <geometry>
-          <mesh filename="package://aero_description/meshes/typeC_lifter/lifter_bone.dae" scale="1 1 1" />
+          <mesh filename="package://noid_description/meshes/typeC_lifter/lifter_bone.dae" scale="1 1 1" />
+        </geometry>
+      </visual>
+      <collision>
+        <origin xyz="0.0 0.0 0" rpy="3.1415 -0 0"/>
+        <geometry>
+          <mesh filename="package://noid_description/meshes/typeC_lifter/lifter_bone.dae" scale="1 1 1" />
         </geometry>
       </collision>
@@ -64,11 +64,11 @@
         <origin xyz="0.0 0.0 0" rpy="3.1415 -0 0"/>
         <geometry>
-          <mesh filename="package://aero_description/meshes/typeC_lifter/lifter_knee.dae" scale="1 1 1" />
-        </geometry>
-      </visual>
-      <collision>
-        <origin xyz="0.0 0.0 0" rpy="3.1415 -0 0"/>
-        <geometry>
-          <mesh filename="package://aero_description/meshes/typeC_lifter/lifter_knee.dae" scale="1 1 1" />
+          <mesh filename="package://noid_description/meshes/typeC_lifter/lifter_knee.dae" scale="1 1 1" />
+        </geometry>
+      </visual>
+      <collision>
+        <origin xyz="0.0 0.0 0" rpy="3.1415 -0 0"/>
+        <geometry>
+          <mesh filename="package://noid_description/meshes/typeC_lifter/lifter_knee.dae" scale="1 1 1" />
         </geometry>
       </collision>
@@ -86,11 +86,11 @@
         <origin xyz="0 0 0.25" rpy="0 0 0"/>
         <geometry>
-          <mesh filename="package://aero_description/meshes/typeC_lifter/lifter_bone.dae" scale="1 1 1" />
-        </geometry>
-      </visual>
-      <collision>
-        <origin xyz="0 0 0.25" rpy="0 0 0"/>
-        <geometry>
-          <mesh filename="package://aero_description/meshes/typeC_lifter/lifter_bone.dae" scale="1 1 1" />
+          <mesh filename="package://noid_description/meshes/typeC_lifter/lifter_bone.dae" scale="1 1 1" />
+        </geometry>
+      </visual>
+      <collision>
+        <origin xyz="0 0 0.25" rpy="0 0 0"/>
+        <geometry>
+          <mesh filename="package://noid_description/meshes/typeC_lifter/lifter_bone.dae" scale="1 1 1" />
         </geometry>
       </collision>
@@ -107,5 +107,5 @@
         <origin xyz="0 0 0.05" rpy="3.1415920 0 0"/>
         <geometry>
-          <mesh filename="package://aero_description/meshes/typeC_lifter/lifter_base.dae" scale="1 1 1" />
+          <mesh filename="package://noid_description/meshes/typeC_lifter/lifter_base.dae" scale="1 1 1" />
         </geometry>
       </visual>
@@ -113,5 +113,5 @@
         <origin xyz="0 0 0.05" rpy="3.1415920 0 0"/>
         <geometry>
-          <mesh filename="package://aero_description/meshes/typeC_lifter/lifter_base.dae" scale="1 1 1" />
+          <mesh filename="package://noid_description/meshes/typeC_lifter/lifter_base.dae" scale="1 1 1" />
         </geometry>
       </collision>
@@ -127,11 +127,11 @@
         <origin xyz="0 0 0" rpy="0 -0 0"/>
         <geometry>
-          <mesh filename="package://aero_description/meshes/typeC_lifter/lifter_top.dae" scale="1 1 1" />
-        </geometry>
-      </visual>
-      <collision>
-        <origin xyz="0 0 0" rpy="0 -0 0"/>
-        <geometry>
-          <mesh filename="package://aero_description/meshes/typeC_lifter/lifter_top.dae" scale="1 1 1" />
+          <mesh filename="package://noid_description/meshes/typeC_lifter/lifter_top.dae" scale="1 1 1" />
+        </geometry>
+      </visual>
+      <collision>
+        <origin xyz="0 0 0" rpy="0 -0 0"/>
+        <geometry>
+          <mesh filename="package://noid_description/meshes/typeC_lifter/lifter_top.dae" scale="1 1 1" />
         </geometry>
       </collision>
@@ -187,5 +187,5 @@
       <visual>
         <geometry>
-          <mesh filename="package://aero_description/meshes/typeC_lifter/lifter_bone_dummy.dae" scale="1 1 1" />
+          <mesh filename="package://noid_description/meshes/typeC_lifter/lifter_bone_dummy.dae" scale="1 1 1" />
         </geometry>
         <origin xyz="0 0 0.25" rpy="0 0 0"/>
@@ -200,5 +200,5 @@
       <visual>
         <geometry>
-          <mesh filename="package://aero_description/meshes/typeC_lifter/lifter_bone_dummy.dae" scale="1 1 1" />
+          <mesh filename="package://noid_description/meshes/typeC_lifter/lifter_bone_dummy.dae" scale="1 1 1" />
         </geometry>
         <origin xyz="0 0 0.25" rpy="0 0 0"/>

File: noid_description/urdf/typeC_lifter/virtual_lifter.urdf.xacro (robot description, xacro)
@@ -14,5 +14,5 @@
        xmlns:physics="http://playerstage.sourceforge.net/gazebo/xmlschema/#physics"
        xmlns:xacro="http://ros.org/wiki/xacro">
-  <xacro:include filename="$(find aero_description)/urdf/common.xacro" />
+  <xacro:include filename="$(find noid_description)/robots/typeF/common.xacro" />
   <xacro:macro name="virtual_lifter" params="base_link x_max x_min z_max z_min">
     <link name="${base_link}" />

File: noid_description/urdf/typeE_wheel/wheels.urdf.xacro (robot description, xacro)
@@ -14,9 +14,9 @@
        xmlns:physics="http://playerstage.sourceforge.net/gazebo/xmlschema/#physics"
        xmlns:xacro="http://ros.org/wiki/xacro">
-  <xacro:include filename="$(find aero_description)/urdf/common.xacro" />
-  <xacro:include filename="$(find aero_description)/common_urdf/gazebo.xacro" />
+  <xacro:include filename="$(find noid_description)/robots/typeF/common.xacro" />
+  <xacro:include filename="$(find noid_description)/urdf/gazebo.xacro" />
   <xacro:property name="wheel_radius" value="0.075"/>
   <xacro:macro name="wheels" params="base_link disable_mesh:=false">
-  <!-- ============================   aero(typeE_wheels)   ============================ -->
+  <!-- ============================   typeE_wheels  ============================ -->
   <link name="${base_link}"/>
     <link name="wheel_base_link">
@@ -24,5 +24,5 @@
         <origin xyz="0.0 0.0 0.0" rpy="0 -0 0"/>
         <geometry>
-          <mesh filename="package://aero_description/meshes/typeE_wheel/wheels_base.dae" scale="1 1 1" />
+          <mesh filename="package://noid_description/meshes/typeE_wheel/wheels_base.dae" scale="1 1 1" />
           </geometry>
       </visual> </xacro:unless>
@@ -30,5 +30,5 @@
         <!--origin xyz="0.0 0.0 0.0" rpy="0 -0 0"/>
         <geometry>
-          <mesh filename="package://aero_description/meshes/typeE_wheel/wheels_base.dae" scale="1 1 1" />
+          <mesh filename="package://noid_description/meshes/typeE_wheel/wheels_base.dae" scale="1 1 1" />
         </geometry-->
         <origin xyz="0.018 0.0 0.0375" rpy="0 -0 0"/>
@@ -48,5 +48,5 @@
         <origin xyz="0.0 0.0 0.0" rpy="0 -0 0"/>
         <geometry>
-          <mesh filename="package://aero_description/meshes/typeE_wheel/wheels_top.dae" scale="1 1 1" />
+          <mesh filename="package://noid_description/meshes/typeE_wheel/wheels_top.dae" scale="1 1 1" />
         </geometry>
       </visual> </xacro:unless>
@@ -63,5 +63,5 @@
         <origin xyz="0.0 0.0 0.0" rpy="-1.57079632679 0 0"/>
         <geometry>
-          <mesh filename="package://aero_description/meshes/typeE_wheel/wheels_mecanum.dae" scale="1 1 1" />
+          <mesh filename="package://noid_description/meshes/typeE_wheel/wheels_mecanum.dae" scale="1 1 1" />
         </geometry>
       </visual> </xacro:unless>
@@ -84,5 +84,5 @@
         <origin xyz="0.0 0.0 0.0" rpy="-1.57079632679 0 0"/>
         <geometry>
-          <mesh filename="package://aero_description/meshes/typeE_wheel/wheels_mecanum.dae" scale="1 1 1" />
+          <mesh filename="package://noid_description/meshes/typeE_wheel/wheels_mecanum.dae" scale="1 1 1" />
         </geometry>
       </visual> </xacro:unless>
@@ -105,5 +105,5 @@
         <origin xyz="0.0 0.0 0.0" rpy="-1.57079632679 0 0"/>
         <geometry>
-          <mesh filename="package://aero_description/meshes/typeE_wheel/wheels_mecanum.dae" scale="1 1 1" />
+          <mesh filename="package://noid_description/meshes/typeE_wheel/wheels_mecanum.dae" scale="1 1 1" />
         </geometry>
       </visual> </xacro:unless>
@@ -126,5 +126,5 @@
         <origin xyz="0.0 0.0 0.0" rpy="-1.57079632679 0 0"/>
         <geometry>
-          <mesh filename="package://aero_description/meshes/typeE_wheel/wheels_mecanum.dae" scale="1 1 1" />
+          <mesh filename="package://noid_description/meshes/typeE_wheel/wheels_mecanum.dae" scale="1 1 1" />
         </geometry>
       </visual> </xacro:unless>
@@ -147,5 +147,5 @@
         <origin xyz="0.0 0.0 0.0" rpy="0 0 0"/>
         <geometry>
-          <mesh filename="package://aero_description/meshes/typeE_wheel/wheels_urg.dae" scale="1 1 1" />
+          <mesh filename="package://noid_description/meshes/typeE_wheel/wheels_urg.dae" scale="1 1 1" />
         </geometry>
       </visual> </xacro:unless>
