Commit message: modify xmlns/property tag of xacro files

File: noid_description/robots/typeF/aero.urdf.xacro (robot description, xacro)
@@ -1,11 +1,5 @@
 <?xml version="1.0"?>
-<robot xmlns:sensor="http://playerstage.sourceforge.net/gazebo/xmlschema/#sensor"
-       xmlns:controller="http://playerstage.sourceforge.net/gazebo/xmlschema/#controller"
-       xmlns:interface="http://playerstage.sourceforge.net/gazebo/xmlschema/#interface"
-       xmlns:xacro="http://playerstage.sourceforge.net/gazebo/xmlschema/#interface"
-       name="SEED-Noid-typeFCET" >
+<robot name="SEED-Noid-typeFCET" xmlns:xacro="http://ros.org/wiki/xacro">
   <!-- The following included files set up definitions of parts of the robot body -->
-  <!-- common variables -->
-  <xacro:include filename="$(find noid_description)/robots/typeF/common.xacro" />
   <!-- wraps upperbody and hand-->
   <xacro:include filename="$(find noid_description)/robots/typeF/noid-upper.urdf.xacro" />

File: noid_description/robots/typeF/noid-upper.urdf.xacro (robot description, xacro)
@@ -1,18 +1,5 @@
 <?xml version="1.0"?>
 <!-- XML namespaces -->
-<robot xmlns:xi="http://www.w3.org/2001/XInclude"
-       xmlns:gazebo="http://playerstage.sourceforge.net/gazebo/xmlschema/#gz"
-       xmlns:model="http://playerstage.sourceforge.net/gazebo/xmlschema/#model"
-       xmlns:sensor="http://playerstage.sourceforge.net/gazebo/xmlschema/#sensor"
-       xmlns:body="http://playerstage.sourceforge.net/gazebo/xmlschema/#body"
-       xmlns:geom="http://playerstage.sourceforge.net/gazebo/xmlschema/#geom"
-       xmlns:joint="http://playerstage.sourceforge.net/gazebo/xmlschema/#joint"
-       xmlns:interface="http://playerstage.sourceforge.net/gazebo/xmlschema/#interface"
-       xmlns:rendering="http://playerstage.sourceforge.net/gazebo/xmlschema/#rendering"
-       xmlns:renderable="http://playerstage.sourceforge.net/gazebo/xmlschema/#renderable"
-       xmlns:controller="http://playerstage.sourceforge.net/gazebo/xmlschema/#controller"
-       xmlns:physics="http://playerstage.sourceforge.net/gazebo/xmlschema/#physics"
-       xmlns:xacro="http://ros.org/wiki/xacro">
-  <xacro:include filename="$(find noid_description)/robots/typeF/common.xacro" />
+<robot name="noid-upper" xmlns:xacro="http://ros.org/wiki/xacro">
   <xacro:include filename="$(find noid_description)/urdf/typeF_upperbody/noid_upper_typef.urdf.xacro" />
   <xacro:include filename="$(find noid_description)/urdf/trx_s/trx_s.urdf.xacro" />

File: noid_description/robots/typeF/noid-wheels.urdf.xacro (robot description, xacro)
@@ -1,18 +1,5 @@
 <?xml version="1.0"?>
 <!-- XML namespaces -->
-<robot xmlns:xi="http://www.w3.org/2001/XInclude"
-       xmlns:gazebo="http://playerstage.sourceforge.net/gazebo/xmlschema/#gz"
-       xmlns:model="http://playerstage.sourceforge.net/gazebo/xmlschema/#model"
-       xmlns:sensor="http://playerstage.sourceforge.net/gazebo/xmlschema/#sensor"
-       xmlns:body="http://playerstage.sourceforge.net/gazebo/xmlschema/#body"
-       xmlns:geom="http://playerstage.sourceforge.net/gazebo/xmlschema/#geom"
-       xmlns:joint="http://playerstage.sourceforge.net/gazebo/xmlschema/#joint"
-       xmlns:interface="http://playerstage.sourceforge.net/gazebo/xmlschema/#interface"
-       xmlns:rendering="http://playerstage.sourceforge.net/gazebo/xmlschema/#rendering"
-       xmlns:renderable="http://playerstage.sourceforge.net/gazebo/xmlschema/#renderable"
-       xmlns:controller="http://playerstage.sourceforge.net/gazebo/xmlschema/#controller"
-       xmlns:physics="http://playerstage.sourceforge.net/gazebo/xmlschema/#physics"
-       xmlns:xacro="http://ros.org/wiki/xacro">
-  <xacro:include filename="$(find noid_description)/robots/typeF/common.xacro" />
+<robot name="noid-whels" xmlns:xacro="http://ros.org/wiki/xacro">
   <xacro:include filename="$(find noid_description)/urdf/typeC_lifter/lifter.urdf.xacro" />
   <xacro:include filename="$(find noid_description)/urdf/typeC_lifter/virtual_lifter.urdf.xacro" />

File: noid_description/urdf/trx_s/trx_s.urdf.xacro (robot description, xacro)
@@ -1,11 +1,7 @@
 <?xml version="1.0"?>
 <!-- XML namespaces -->
-<robot xmlns:sensor="http://playerstage.sourceforge.net/gazebo/xmlschema/#sensor"
-       xmlns:controller="http://playerstage.sourceforge.net/gazebo/xmlschema/#controller"
-       xmlns:interface="http://playerstage.sourceforge.net/gazebo/xmlschema/#interface"
-       xmlns:xacro="http://ros.org/wiki/xacro">
-  <xacro:include filename="$(find noid_description)/robots/typeF/common.xacro" />
+<robot name="trx_s" xmlns:xacro="http://ros.org/wiki/xacro">
+  <xacro:property name="M_PI" value="3.1415926535897931" />
   <xacro:include filename="$(find noid_description)/urdf/gazebo.xacro" />
-  <property name="M_PI" value="3.1415926535897931" />
   <xacro:macro name="trx_s" params="prefix:=r reflect:=1 disable_mesh:=false">
   <!-- ============================   Hand(trx_s)   ============================ -->

File: noid_description/urdf/typeC_lifter/lifter.urdf.xacro (robot description, xacro)
@@ -1,18 +1,5 @@
 <?xml version="1.0"?>
 <!-- XML namespaces -->
-<robot xmlns:xi="http://www.w3.org/2001/XInclude"
-       xmlns:gazebo="http://playerstage.sourceforge.net/gazebo/xmlschema/#gz"
-       xmlns:model="http://playerstage.sourceforge.net/gazebo/xmlschema/#model"
-       xmlns:sensor="http://playerstage.sourceforge.net/gazebo/xmlschema/#sensor"
-       xmlns:body="http://playerstage.sourceforge.net/gazebo/xmlschema/#body"
-       xmlns:geom="http://playerstage.sourceforge.net/gazebo/xmlschema/#geom"
-       xmlns:joint="http://playerstage.sourceforge.net/gazebo/xmlschema/#joint"
-       xmlns:interface="http://playerstage.sourceforge.net/gazebo/xmlschema/#interface"
-       xmlns:rendering="http://playerstage.sourceforge.net/gazebo/xmlschema/#rendering"
-       xmlns:renderable="http://playerstage.sourceforge.net/gazebo/xmlschema/#renderable"
-       xmlns:controller="http://playerstage.sourceforge.net/gazebo/xmlschema/#controller"
-       xmlns:physics="http://playerstage.sourceforge.net/gazebo/xmlschema/#physics"
-       xmlns:xacro="http://ros.org/wiki/xacro">
-  <xacro:include filename="$(find noid_description)/robots/typeF/common.xacro" />
+<robot name="lifter" xmlns:xacro="http://ros.org/wiki/xacro">
   <xacro:include filename="$(find noid_description)/urdf/gazebo.xacro" />
   <xacro:macro name="lifter" params="base_link">

File: noid_description/urdf/typeC_lifter/virtual_lifter.urdf.xacro (robot description, xacro)
@@ -1,18 +1,5 @@
 <?xml version="1.0"?>
 <!-- XML namespaces -->
-<robot xmlns:xi="http://www.w3.org/2001/XInclude"
-       xmlns:gazebo="http://playerstage.sourceforge.net/gazebo/xmlschema/#gz"
-       xmlns:model="http://playerstage.sourceforge.net/gazebo/xmlschema/#model"
-       xmlns:sensor="http://playerstage.sourceforge.net/gazebo/xmlschema/#sensor"
-       xmlns:body="http://playerstage.sourceforge.net/gazebo/xmlschema/#body"
-       xmlns:geom="http://playerstage.sourceforge.net/gazebo/xmlschema/#geom"
-       xmlns:joint="http://playerstage.sourceforge.net/gazebo/xmlschema/#joint"
-       xmlns:interface="http://playerstage.sourceforge.net/gazebo/xmlschema/#interface"
-       xmlns:rendering="http://playerstage.sourceforge.net/gazebo/xmlschema/#rendering"
-       xmlns:renderable="http://playerstage.sourceforge.net/gazebo/xmlschema/#renderable"
-       xmlns:controller="http://playerstage.sourceforge.net/gazebo/xmlschema/#controller"
-       xmlns:physics="http://playerstage.sourceforge.net/gazebo/xmlschema/#physics"
-       xmlns:xacro="http://ros.org/wiki/xacro">
-  <xacro:include filename="$(find noid_description)/robots/typeF/common.xacro" />
+<robot name="virtual_lifter" xmlns:xacro="http://ros.org/wiki/xacro">
   <xacro:macro name="virtual_lifter" params="base_link x_max x_min z_max z_min">
     <link name="${base_link}" />

File: noid_description/urdf/typeE_wheel/wheels.urdf.xacro (robot description, xacro)
@@ -1,18 +1,5 @@
 <?xml version="1.0"?>
 <!-- XML namespaces -->
-<robot xmlns:xi="http://www.w3.org/2001/XInclude"
-       xmlns:gazebo="http://playerstage.sourceforge.net/gazebo/xmlschema/#gz"
-       xmlns:model="http://playerstage.sourceforge.net/gazebo/xmlschema/#model"
-       xmlns:sensor="http://playerstage.sourceforge.net/gazebo/xmlschema/#sensor"
-       xmlns:body="http://playerstage.sourceforge.net/gazebo/xmlschema/#body"
-       xmlns:geom="http://playerstage.sourceforge.net/gazebo/xmlschema/#geom"
-       xmlns:joint="http://playerstage.sourceforge.net/gazebo/xmlschema/#joint"
-       xmlns:interface="http://playerstage.sourceforge.net/gazebo/xmlschema/#interface"
-       xmlns:rendering="http://playerstage.sourceforge.net/gazebo/xmlschema/#rendering"
-       xmlns:renderable="http://playerstage.sourceforge.net/gazebo/xmlschema/#renderable"
-       xmlns:controller="http://playerstage.sourceforge.net/gazebo/xmlschema/#controller"
-       xmlns:physics="http://playerstage.sourceforge.net/gazebo/xmlschema/#physics"
-       xmlns:xacro="http://ros.org/wiki/xacro">
-  <xacro:include filename="$(find noid_description)/robots/typeF/common.xacro" />
+<robot name="wheels" xmlns:xacro="http://ros.org/wiki/xacro">
   <xacro:include filename="$(find noid_description)/urdf/gazebo.xacro" />
   <xacro:property name="wheel_radius" value="0.075"/>

File: noid_description/urdf/typeF_upperbody/noid_upper_typef.urdf.xacro (robot description, xacro)
@@ -1,9 +1,5 @@
 <?xml version="1.0"?>
 <!-- XML namespaces -->
-<robot xmlns:sensor="http://playerstage.sourceforge.net/gazebo/xmlschema/#sensor"
-       xmlns:controller="http://playerstage.sourceforge.net/gazebo/xmlschema/#controller"
-       xmlns:interface="http://playerstage.sourceforge.net/gazebo/xmlschema/#interface"
-       xmlns:xacro="http://ros.org/wiki/xacro">
-  <xacro:include filename="$(find noid_description)/robots/typeF/common.xacro" />
+<robot name="noid_upper_typef" xmlns:xacro="http://ros.org/wiki/xacro">
   <xacro:include filename="$(find noid_description)/urdf/gazebo.xacro" />
   <xacro:property name="wrist_sensor_offset" value="0.0"/>
