Commit message: added typefcety and fcesy

File: seed_r7_description/typefcesy/noid-upper.urdf.xacro (robot description, xacro)
@@ -3,5 +3,5 @@
 <robot name="noid-upper" xmlns:xacro="http://ros.org/wiki/xacro">
   <xacro:include filename="$(find seed_r7_description)/urdf/typeF_upperbody/noid_upper_typef.urdf.xacro" />
-  <xacro:include filename="$(find seed_r7_description)/urdf/trx_s/trx_s.urdf.xacro" />
+  <xacro:include filename="$(find seed_r7_description)/urdf/seed_hand/seed_hand.urdf.xacro" />
   <xacro:include filename="$(find seed_r7_description)/urdf/hand_yaw/hand_yaw.urdf.xacro" />
   <xacro:macro name="noid-upper" params="disable_mesh:=false">
@@ -9,15 +9,15 @@
   <xacro:hand_yaw prefix="r" reflect="1" wrist_link="r_wrist_top" disable_mesh="${disable_mesh}"/>
   <xacro:hand_yaw prefix="l" reflect="-1" wrist_link="l_wrist_top" disable_mesh="${disable_mesh}"/>
-  <xacro:trx_s prefix="r" reflect="1" disable_mesh="${disable_mesh}"/>
-  <xacro:trx_s prefix="l" reflect="-1" disable_mesh="${disable_mesh}"/>
+  <xacro:seed_hand prefix="r" reflect="1" disable_mesh="${disable_mesh}"/>
+  <xacro:seed_hand prefix="l" reflect="-1" disable_mesh="${disable_mesh}"/>
   <joint name="r_hand_connector" type="fixed">
     <parent link="r_hand_yaw_link"/>
     <child link="r_hand_link"/>
-    <origin xyz="0.0 0.0 -0.02" rpy="0 0 0 "/>
+    <origin xyz="0.0 0.0 -0.01" rpy="0 0 0 "/>
   </joint>
   <joint name="l_hand_connector" type="fixed">
     <parent link="l_hand_yaw_link"/>
     <child link="l_hand_link"/>
-    <origin xyz="0.0 0.0 -0.02" rpy="0 0 0 "/>
+    <origin xyz="0.0 0.0 -0.01" rpy="0 0 0 "/>
   </joint>
   <joint name="upper_lower_connector" type="fixed">

File: seed_r7_description/urdf/typeF_upperbody/noid_upper_typef.urdf.xacro (robot description, xacro)
@@ -190,10 +190,4 @@
   <xacro:gazebo_link_reference link_name="l_forearm_link" />
   <link name="l_wrist_center">
-  <xacro:unless value="${disable_mesh}"> <visual>
-      <origin xyz="0 0 0" rpy="0 1.57 1.57"/>
-      <geometry>
-        <mesh filename="package://seed_r7_description/meshes/typeF_upperbody/wrist.dae" scale="1 1 1" />
-      </geometry>
-    </visual> </xacro:unless>
     <inertial>
       <mass value="0.05" />
@@ -204,4 +198,16 @@
   <xacro:gazebo_link_reference link_name="l_wrist_center" />
   <link name="l_wrist_top">
+   <xacro:unless value="${disable_mesh}"> <visual>
+      <origin xyz="0 0 0" rpy="0 1.57 1.57"/>
+      <geometry>
+        <mesh filename="package://seed_r7_description/meshes/typeF_upperbody/wrist.dae" scale="1 1 1" />
+      </geometry>
+    </visual> </xacro:unless>
+    <xacro:unless value="${disable_mesh}"> <collision>
+      <origin xyz="0 0 0" rpy="0 1.57 1.57"/>
+      <geometry>
+        <mesh filename="package://seed_r7_description/meshes/typeF_upperbody/wrist.dae" scale="1 1 1" />
+      </geometry>
+    </collision> </xacro:unless>
     <inertial>
       <mass value="0.05" />
