Commit message: updated typefcesy and fcety noid.urdf

File: seed_r7_description/typefcesy/noid.urdf (robot description, URDF)
Before this commit: robot SEED-Noid-Mover-typeFCESy, 59 links, 58 joints
Links:
- link l_hand_yaw_link: geometry collision cylinder length=0.01 radius=0.03; visual mesh filename=package://seed_r7_description/meshes/hand_yaw/hand_yaw.dae scale=1 1 1
- link l_wrist_center: geometry 
- link l_wrist_top: geometry collision mesh filename=package://seed_r7_description/meshes/typeF_upperbody/wrist.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 scale=1 1 1; visual mesh filename=package://seed_r7_description/meshes/typeF_upperbody/wrist.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 scale=1 1 1
- link r_hand_yaw_link: geometry collision cylinder length=0.01 radius=0.03; visual mesh filename=package://seed_r7_description/meshes/hand_yaw/hand_yaw.dae scale=1 1 1

File: seed_r7_description/typefcety/noid.urdf (robot description, URDF)
Before this commit: robot SEED-Noid-Mover-typeFCETy, 55 links, 54 joints
Links:
- removed link l_eef_pick_link
- removed link l_index_tip_link
- removed link l_thumb_tip_link
- removed link r_eef_pick_link
- removed link r_index_tip_link
- removed link r_thumb_tip_link
- added link l_hand_yaw_link, mass 0.183; collision cylinder length=0.01 radius=0.03; visual mesh filename=package://seed_r7_description/meshes/hand_yaw/hand_yaw.dae scale=1 1 1
- added link l_wrist_top, mass 0.05; collision mesh filename=package://seed_r7_description/meshes/typeF_upperbody/wrist.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 scale=1 1 1; visual mesh filename=package://seed_r7_description/meshes/typeF_upperbody/wrist.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 scale=1 1 1
- added link r_hand_yaw_link, mass 0.183; collision cylinder length=0.01 radius=0.03; visual mesh filename=package://seed_r7_description/meshes/hand_yaw/hand_yaw.dae scale=1 1 1
- added link r_wrist_top, mass 0.05; collision mesh filename=package://seed_r7_description/meshes/typeF_upperbody/wrist.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 scale=1 1 1; visual mesh filename=package://seed_r7_description/meshes/typeF_upperbody/wrist.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 scale=1 1 1
- link l_hand_link: geometry collision box size=0.036 0.050 0.070; collision box size=0.036 0.070 0.030
- link l_indexbase_link: geometry collision box size=0.041 0.061 0.010; visual mesh filename=package://seed_r7_description/meshes/trx_s/index_base.DAE
- link l_indexend_link: geometry collision box size=0.040 0.028 0.016; visual mesh filename=package://seed_r7_description/meshes/trx_s/index_end.DAE
- link l_indexmid_link: geometry collision box size=0.034 0.030 0.010; visual mesh filename=package://seed_r7_description/meshes/trx_s/index_mid.DAE
- link l_thumb_link: geometry collision box size=0.012 0.008 0.050; collision box size=0.012 0.008 0.050
- link r_hand_link: geometry collision box size=0.036 0.050 0.070; collision box size=0.036 0.070 0.030
- link r_indexbase_link: geometry collision box size=0.041 0.061 0.010; visual mesh filename=package://seed_r7_description/meshes/trx_s/index_base.DAE
- link r_indexend_link: geometry collision box size=0.040 0.028 0.016; visual mesh filename=package://seed_r7_description/meshes/trx_s/index_end.DAE
- link r_indexmid_link: geometry collision box size=0.034 0.030 0.010; visual mesh filename=package://seed_r7_description/meshes/trx_s/index_mid.DAE
- link r_thumb_link: geometry collision box size=0.012 0.008 0.050; collision box size=0.012 0.008 0.050
Joints:
- removed joint l_eef_pick_joint
- removed joint l_index_tip_joint
- removed joint l_thumb_tip_joint
- removed joint r_eef_pick_joint
- removed joint r_index_tip_joint
- removed joint r_thumb_tip_joint
- added joint l_hand_connector: type fixed, parent l_hand_yaw_link, child l_hand_link, origin xyz=0.0 0.0 -0.01 rpy=0 0 0 
- added joint l_hand_y_joint: type revolute, parent l_wrist_top, child l_hand_yaw_link, origin xyz=0 0 -0.031 rpy=0 0 0, axis 0 0 1, limit lower=-2.0 upper=2.0 effort=100 velocity=3.1
- added joint r_hand_connector: type fixed, parent r_hand_yaw_link, child r_hand_link, origin xyz=0.0 0.0 -0.01 rpy=0 0 0 
- added joint r_hand_y_joint: type revolute, parent r_wrist_top, child r_hand_yaw_link, origin xyz=0 0 -0.031 rpy=0 0 0, axis 0 0 1, limit lower=-2.0 upper=2.0 effort=100 velocity=3.1
- joint l_indexbase_joint: limit lower=-3.14159 upper=3.14159 effort=100 velocity=0.5 -> lower=-3.14159 upper=3.14159 effort=25 velocity=0.5; origin xyz=0 0.013 -0.115 rpy=0 -0 0  -> xyz=0 0.013 -0.087 rpy=0.3 0 0; type revolute -> continuous
- joint l_indexend_joint: limit lower=-3.14159 upper=3.14159 effort=100 velocity=0.5 -> lower=-3.14159 upper=3.14159 effort=25 velocity=0.5; origin xyz=0 -0.021716 -0.013357 rpy=0 -0 0  -> xyz=0 0.005 -0.025 rpy=1.13 0 0 ; type revolute -> continuous
- joint l_indexmid_joint: limit lower=-3.14159 upper=3.14159 effort=100 velocity=0.5 -> lower=-3.14159 upper=3.14159 effort=25 velocity=0.5; origin xyz=0 -0.028754 -0.034615 rpy=0 -0 0  -> xyz=0 0 -0.045 rpy=-0.52 0 0 ; type revolute -> continuous
- joint l_thumb_joint: limit lower=-3.14159 upper=3.14159 effort=100 velocity=0.5 -> lower=-0.0 upper=1.57 effort=25 velocity=0.5; origin xyz=0 -0.022355 -0.079645 rpy=0 -0 0  -> xyz=0 -0.023 -0.054 rpy=0.08  0 0
- joint l_wrist_r_joint: child l_hand_link -> l_wrist_top
- joint r_indexbase_joint: limit lower=-3.14159 upper=3.14159 effort=100 velocity=0.5 -> lower=-3.14159 upper=3.14159 effort=25 velocity=0.5; origin xyz=0 -0.013 -0.115 rpy=0 -0 0  -> xyz=0 -0.013 -0.087 rpy=-0.3 0 0; type revolute -> continuous
- joint r_indexend_joint: limit lower=-3.14159 upper=3.14159 effort=100 velocity=0.5 -> lower=-3.14159 upper=3.14159 effort=25 velocity=0.5; origin xyz=0 0.021716 -0.013357 rpy=0 -0 0  -> xyz=0 -0.005 -0.025 rpy=-1.13 0 0 ; type revolute -> continuous
- joint r_indexmid_joint: limit lower=-3.14159 upper=3.14159 effort=100 velocity=0.5 -> lower=-3.14159 upper=3.14159 effort=25 velocity=0.5; origin xyz=0 0.028754 -0.034615 rpy=0 -0 0  -> xyz=0 0 -0.045 rpy=0.52 0 0 ; type revolute -> continuous
- joint r_thumb_joint: limit lower=-3.14159 upper=3.14159 effort=100 velocity=0.5 -> lower=-1.57 upper=0.0 effort=25 velocity=0.5; origin xyz=0 0.022355 -0.079645 rpy=0 -0 0  -> xyz=0 0.023 -0.054 rpy=-0.08  0 0
- joint r_wrist_r_joint: child r_hand_link -> r_wrist_top
