Commit message: divided hand model added

File: seed_r7_description/urdf/hand_yaw/hand_yaw.urdf.xacro (robot description, xacro)
@@ -4,5 +4,5 @@
   <xacro:property name="M_PI" value="3.1415926535897931" />
   <xacro:include filename="$(find seed_r7_description)/urdf/gazebo.xacro" />
-  <xacro:macro name="hand_yaw" params="prefix:=r reflect:=1 hand_link disable_mesh:=false">
+  <xacro:macro name="hand_yaw" params="prefix:=r reflect:=1 wrist_link disable_mesh:=false">
   <!-- ============================   hand_yaw   ============================ -->
     <!-- prefix is "r" or "l" -->
@@ -10,15 +10,9 @@
   <link name="${prefix}_hand_yaw_link">
     <xacro:unless value="${disable_mesh}"> <visual>
-      <origin xyz="0.0 0 0" rpy="0 ${M_PI / 2.0} ${reflect * M_PI / 2.0}"/>
+      <origin xyz="0.0 0 0.0" rpy="0 3.14 3.14"/>
       <geometry>
-        <mesh filename="package://seed_r7_description/meshes/hand_yaw/wrist.dae" scale="1 1 1" />
+        <mesh filename="package://seed_r7_description/meshes/hand_yaw/hand_yaw.dae" scale="1 1 1" />
       </geometry>
     </visual> </xacro:unless>
-    <xacro:unless value="${disable_mesh}"> <collision>
-      <origin xyz="0 0 0" rpy="0 ${M_PI / 2.0} ${reflect * M_PI / 2.0}"/>
-      <geometry>
-        <mesh filename="package://seed_r7_description/meshes/hand_yaw/wrist.dae" scale="1 1 1" />
-      </geometry>
-    </collision> </xacro:unless>
     <inertial>
       <mass value="0.183" />
@@ -36,7 +30,7 @@
   </gazebo>
   <joint name="${prefix}_hand_y_joint" type="revolute">
-    <parent link="${prefix}_hand_yaw_link"/>
-    <child  link="${hand_link}"/>
-    <origin xyz="0 0 -0.04" rpy="0 0 0"/>
+    <parent link="${wrist_link}"/>
+    <child  link="${prefix}_hand_yaw_link"/>
+    <origin xyz="0 0 -0.031" rpy="0 0 0"/>
     <axis   xyz="0 0 1"/>
     <limit lower="-2.0" upper="2.0" effort="100" velocity="3.1" />

File: seed_r7_description/urdf/trx_s/trx_s.urdf.xacro (robot description, xacro)
@@ -1,173 +1,81 @@
 <?xml version="1.0"?>
-<!-- XML namespaces -->
 <robot name="trx_s" xmlns:xacro="http://ros.org/wiki/xacro">
-  <xacro:property name="M_PI" value="3.1415926535897931" />
-  <xacro:include filename="$(find seed_r7_description)/urdf/gazebo.xacro" />
-  <xacro:macro name="trx_s" params="prefix:=r reflect:=1 disable_mesh:=false">
-  <!-- ============================   Hand(trx_s)   ============================ -->
-    <!-- prefix is "r" or "l" -->
-    <!-- reflect=1 is rightside, reflect=-1 is leftside -->
+<xacro:property name="M_PI" value="3.1415926535897931" />
+<xacro:macro name="trx_s" params="prefix:=r reflect:=1 disable_mesh:=false">
+<!-- hand -->
   <link name="${prefix}_hand_link">
-    <xacro:unless value="${disable_mesh}"> <visual>
-      <origin xyz="0 0 0" rpy="0 -0 ${(1.0 - reflect) * M_PI / 2.0}"/>
+    <visual>
       <geometry>
-        <mesh filename="package://seed_r7_description/meshes/trx_s/RARM_LINK7_mesh.dae" scale="1 1 1" />
+        <mesh filename="package://seed_r7_description/meshes/trx_s/hand.DAE"/>
       </geometry>
-    </visual> </xacro:unless>
-    <xacro:unless value="${disable_mesh}">
-    <collision>
-      <origin rpy="${reflect * 0.7} 0 0" xyz="0 0 -0.093"/>
+      <origin xyz="0 0 0" rpy="${M_PI} 0 ${reflect * M_PI / 2.0}"/>
+    </visual>
+  </link>
+<!-- hand index base -->
+  <link name="${prefix}_indexbase_link">
+    <visual>
       <geometry>
-        <box size="0.036 0.070 0.030" />
+        <mesh filename="package://seed_r7_description/meshes/trx_s/index_base.DAE"/>
       </geometry>
-    </collision>
-    <collision>
-      <origin rpy="${reflect * -0.10} 0 0" xyz="0 ${reflect * -0.007} -0.055"/>
-      <geometry>
-        <box size="0.036 0.050 0.070" />
-      </geometry>
-    </collision>
-    </xacro:unless>
-    <inertial>
-      <mass value="0.183" />
-      <origin xyz="0 0 -0.0875" rpy="0 -0 0"/>
-      <inertia ixx="0.000601" ixy="0" ixz="0" iyy="0.00055" iyz="0" izz="0.000102"/>
-    </inertial>
+      <origin xyz="0 0 0" rpy="${M_PI} 0 ${reflect * M_PI / 2.0}"/>
+    </visual>
   </link>
-  <xacro:gazebo_link_reference link_name="${prefix}_hand_link" />
-  <link name="${prefix}_indexbase_link">
-    <xacro:unless value="${disable_mesh}"> <visual>
-      <origin xyz="0 ${0.013 * reflect} 0.115" rpy="0 -0 ${(1.0 - reflect) * M_PI / 2.0}"/>
-      <geometry>
-        <mesh filename="package://seed_r7_description/meshes/trx_s/RARM_INDEX_LINK1_mesh.dae" scale="1 1 1" />
-      </geometry>
-    </visual> </xacro:unless>
-    <xacro:unless value="${disable_mesh}"> <collision>
-      <origin xyz="0 ${reflect * 0.013494 } -0.021422" rpy="${reflect * -0.85} 0 0"/>
-      <geometry>
-        <box size="0.041 0.061 0.016" />  <!-- 0.85 -->
-      </geometry>
-    </collision> </xacro:unless>
-    <inertial>
-      <mass value="0.1" />
-      <origin xyz="0 ${reflect * 0.014} -0.021" rpy="0 0 0"/>
-      <inertia ixx="0.001" iyy="0.0001" izz="0.0001" ixy="0" ixz="0" iyz="0" />
-    </inertial>
-  </link>
-  <xacro:gazebo_link_reference link_name="${prefix}_indexbase_link" />
-  <link name="${prefix}_indexmid_link">
-    <xacro:unless value="${disable_mesh}"> <visual>
-      <origin xyz="0 ${-0.015754 * reflect} 0.149615" rpy="0 -0 ${(1.0 - reflect) * M_PI / 2.0}"/>
-      <geometry>
-        <mesh filename="package://seed_r7_description/meshes/trx_s/RARM_INDEX_LINK2_mesh.dae" scale="1 1 1" />
-      </geometry>
-    </visual> </xacro:unless>
-    <xacro:unless value="${disable_mesh}"> <collision>
-      <origin xyz="0 ${reflect * 0.014} -0.008" rpy="${reflect * -0.3} 0 0"/> <!-- 0.3 -->
-      <geometry>
-        <box size="0.034 0.030 0.016" />
-      </geometry>
-    </collision> </xacro:unless>
-    <inertial>
-      <mass value="0.1" />
-      <origin xyz="0 ${reflect * 0.014} -0.008" rpy="0 0 0"/>
-      <inertia ixx="0.001" iyy="0.0001" izz="0.0001" ixy="0" ixz="0" iyz="0" />
-    </inertial>
-  </link>
-  <xacro:gazebo_link_reference link_name="${prefix}_indexmid_link" />
-  <link name="${prefix}_indexend_link">
-    <xacro:unless value="${disable_mesh}"> <visual>
-      <origin xyz="0 ${-0.03747 * reflect} 0.162972" rpy="0 -0 ${(1.0 - reflect) * M_PI / 2.0}"/>
-      <geometry>
-        <mesh filename="package://seed_r7_description/meshes/trx_s/RARM_INDEX_LINK3_mesh.dae" scale="1 1 1" />
-      </geometry>
-    </visual> </xacro:unless>
-    <xacro:unless value="${disable_mesh}"> <collision>
-      <origin xyz="0 ${reflect * 0.013} 0.004" rpy="0 0 0"/> <!-- 0.0 -->
-      <geometry>
-        <box size="0.040 0.028 0.016" />
-      </geometry>
-    </collision> </xacro:unless>
-    <inertial>
-      <mass value="0.1" />
-      <origin xyz="0 ${reflect * 0.02} 0" rpy="0 0 0"/>
-      <inertia ixx="0.0001" iyy="0.0001" izz="0.0001" ixy="0" ixz="0" iyz="0" />
-    </inertial>
-  </link>
-  <xacro:gazebo_link_reference link_name="${prefix}_indexend_link" />
-  <link name="${prefix}_thumb_link">
-    <xacro:unless value="${disable_mesh}"> <visual>
-      <origin xyz="0 ${-0.022355 * reflect} 0.079645" rpy="0 -0 ${(1.0 - reflect) * M_PI / 2.0}"/>
-      <geometry>
-        <mesh filename="package://seed_r7_description/meshes/trx_s/RARM_THUMB_LINK_mesh.dae" scale="1 1 1" />
-      </geometry>
-    </visual> </xacro:unless>
-    <xacro:unless value="${disable_mesh}">
-    <collision>
-      <origin rpy="${reflect * 0.63} 0 0" xyz="0.0 ${reflect * 0.019645} -0.010355"/>
-      <geometry>
-        <box size="0.012 0.008 0.050"/>
-      </geometry>
-    </collision>
-    <collision>
-      <origin rpy="${reflect * 0.1} 0 0" xyz="0.0 ${reflect * 0.035645} -0.050355"/>
-      <geometry>
-        <box size="0.012 0.008 0.050"/>
-      </geometry>
-    </collision>
-    </xacro:unless>
-    <inertial>
-      <mass value="0.1" />
-      <origin xyz="0 ${reflect * 0.05} -0.06" rpy="0 0 0"/>
-      <inertia ixx="0.001" iyy="0.0001" izz="0.0001" ixy="0" ixz="0" iyz="0" />
-    </inertial>
-  </link>
-  <xacro:gazebo_link_reference link_name="${prefix}_thumb_link" />
-  <joint name="${prefix}_indexbase_joint" type="revolute">
+  <joint name="${prefix}_indexbase_joint" type="continuous">
     <parent link="${prefix}_hand_link"/>
     <child  link="${prefix}_indexbase_link"/>
-    <origin xyz="0 ${-0.013 * reflect} -0.115" rpy="0 -0 0 "/>
+    <origin xyz="0 ${-0.013*reflect} -0.087" rpy="0 0 0"/>
     <axis   xyz="1 0 0"/>
-    <limit lower="-3.14159" upper="3.14159" effort="100" velocity="0.5" />
-    <dynamics damping="0.2" friction="0" />
+    <limit lower="-3.14159" upper="3.14159" effort="25" velocity="0.5" />
   </joint>
-  <!--xacro:gazebo_joint_reference joint_name="${prefix}_indexbase_joint" /-->
-  <xacro:gazebo_transmission joint_name="${prefix}_indexbase_joint" />
-  <joint name="${prefix}_indexmid_joint" type="revolute">
+<!-- hand index middle -->
+  <link name="${prefix}_indexmid_link">
+    <visual>
+      <geometry>
+        <mesh filename="package://seed_r7_description/meshes/trx_s/index_mid.DAE"/>
+      </geometry>
+      <origin xyz="0 0 0" rpy="${M_PI} 0 ${reflect * M_PI / 2.0}"/>
+    </visual>
+  </link>
+  <joint name="${prefix}_indexmid_joint" type="continuous">
     <parent link="${prefix}_indexbase_link"/>
     <child  link="${prefix}_indexmid_link"/>
-    <origin xyz="0 ${0.028754 * reflect} -0.034615" rpy="0 -0 0 "/>
+    <origin xyz="0 0 -0.045" rpy="${0.52*reflect} 0 0 "/>
     <axis   xyz="1 0 0"/>
-    <limit lower="-3.14159" upper="3.14159" effort="100" velocity="0.5" />
-    <dynamics damping="0.2" friction="0" />
+    <limit lower="-3.14159" upper="3.14159" effort="25" velocity="0.5" />
   </joint>
-  <!--xacro:gazebo_joint_reference joint_name="${prefix}_indexmid_joint" /-->
-  <xacro:gazebo_transmission joint_name="${prefix}_indexmid_joint" />
-  <joint name="${prefix}_indexend_joint" type="revolute">
+<!-- hand index end -->
+  <link name="${prefix}_indexend_link">
+    <visual>
+      <geometry>
+        <mesh filename="package://seed_r7_description/meshes/trx_s/index_end.DAE"/>
+      </geometry>
+      <origin xyz="0 0 0" rpy="${M_PI} 0 ${reflect * M_PI / 2.0}"/>
+    </visual>
+  </link>
+  <joint name="${prefix}_indexend_joint" type="continuous">
     <parent link="${prefix}_indexmid_link"/>
     <child  link="${prefix}_indexend_link"/>
-    <origin xyz="0 ${0.021716 * reflect} -0.013357" rpy="0 -0 0 "/>
+    <origin xyz="0 ${-0.005*reflect} -0.025" rpy="${-1.13*reflect} 0 0 "/>
     <axis   xyz="1 0 0"/>
-    <limit lower="-3.14159" upper="3.14159" effort="100" velocity="0.5" />
-    <dynamics damping="0.2" friction="0" />
+    <limit lower="-3.14159" upper="3.14159" effort="25" velocity="0.5" />
   </joint>
-  <!--xacro:gazebo_joint_reference joint_name="${prefix}_indexend_joint" /-->
-  <xacro:gazebo_transmission joint_name="${prefix}_indexend_joint" />
+<!-- hand finger -->
+  <link name="${prefix}_thumb_link">
+    <visual>
+      <geometry>
+        <mesh filename="package://seed_r7_description/meshes/trx_s/thumb.DAE"/>
+      </geometry>
+      <origin xyz="0 0 0" rpy="${M_PI} 0 ${reflect * M_PI / 2.0}"/>
+    </visual>
+  </link>
   <joint name="${prefix}_thumb_joint" type="revolute">
-    <parent link="${prefix}_hand_link"/>
+    <parent  link="${prefix}_hand_link"/>
     <child  link="${prefix}_thumb_link"/>
-    <origin xyz="0 ${0.022355 * reflect} -0.079645" rpy="0 -0 0 "/>
+    <origin xyz="0 ${0.023*reflect} -0.054" rpy="${-0.08 * reflect}  0 0"/>
     <axis   xyz="1 0 0"/>
-    <limit lower="-3.14159" upper="3.14159" effort="100" velocity="0.5" />
-    <dynamics damping="0.2" friction="0" />
+    <limit lower="${-1.57 * (1 + reflect)/2.0}" upper="${1.57 * (1 - reflect)/2.0}" effort="25" velocity="0.5" />
   </joint>
-  <xacro:gazebo_transmission joint_name="${prefix}_thumb_joint" />
-  <!-- for ik eef link-->
   <link name="${prefix}_eef_grasp_link"/>
-  <link name="${prefix}_eef_pick_link"/>
-  <link name="${prefix}_thumb_tip_link"/>
-  <link name="${prefix}_index_tip_link"/>
-  <!-- for ik eef link-->
-  <!-- for ik eef connector-->
+   <!-- for ik eef connector-->
   <joint name="${prefix}_eef_grasp_joint" type="fixed">
     <parent  link="${prefix}_hand_link"/>
@@ -175,20 +83,4 @@
     <origin xyz="0.0 ${0.04 * reflect} -0.14" rpy="0 1.5708 0 "/>
   </joint>
-  <joint name="${prefix}_eef_pick_joint" type="fixed">
-    <parent  link="${prefix}_hand_link"/>
-    <child link="${prefix}_eef_pick_link"/>
-    <origin xyz="0.0 ${0.07 * reflect} -0.16" rpy="0 1.5708 0 "/>
-  </joint>
-  <joint name="${prefix}_thumb_tip_joint" type="fixed">
-    <parent  link="${prefix}_thumb_link"/>
-    <child link="${prefix}_thumb_tip_link"/>
-    <origin xyz="0.0 ${0.035 * reflect} -0.085" rpy="0 0 0 "/>
-  </joint>
-  <joint name="${prefix}_index_tip_joint" type="fixed">
-    <parent  link="${prefix}_indexend_link"/>
-    <child link="${prefix}_index_tip_link"/>
-    <origin xyz="0.0 ${0.02 * reflect} 0.0" rpy="0 0 0 "/>
-  </joint>
-  <!-- for ik eef connector-->
   </xacro:macro>
 </robot>

File: seed_r7_description/urdf/typeF_upperbody/noid_upper_typef.urdf.xacro (robot description, xacro)
@@ -197,4 +197,23 @@
   </link>
   <xacro:gazebo_link_reference link_name="l_wrist_center" />
+  <link name="l_wrist_top">
+   <xacro:unless value="${disable_mesh}"> <visual>
+      <origin xyz="0 0 0" rpy="0 1.57 1.57"/>
+      <geometry>
+        <mesh filename="package://seed_r7_description/meshes/typeF_upperbody/wrist.dae" scale="1 1 1" />
+      </geometry>
+    </visual> </xacro:unless>
+    <xacro:unless value="${disable_mesh}"> <collision>
+      <origin xyz="0 0 0" rpy="0 1.57 1.57"/>
+      <geometry>
+        <mesh filename="package://seed_r7_description/meshes/typeF_upperbody/wrist.dae" scale="1 1 1" />
+      </geometry>
+    </collision> </xacro:unless>
+    <inertial>
+      <mass value="0.05" />
+      <origin xyz="0 0 0" rpy="0 -0 0"/>
+      <inertia ixx="0.0001" ixy="0" ixz="0" iyy="0.0001" iyz="0" izz="0.0001"/>
+    </inertial>
+  </link>
   <link name="neck_link">
     <xacro:unless value="${disable_mesh}"> <visual>
@@ -376,4 +395,23 @@
   </link>
   <xacro:gazebo_link_reference link_name="r_wrist_center" />
+  <link name="r_wrist_top">
+   <xacro:unless value="${disable_mesh}"> <visual>
+      <origin xyz="0 0 0" rpy="0 1.57 1.57"/>
+      <geometry>
+        <mesh filename="package://seed_r7_description/meshes/typeF_upperbody/wrist.dae" scale="1 1 1" />
+      </geometry>
+    </visual> </xacro:unless>
+    <xacro:unless value="${disable_mesh}"> <collision>
+      <origin xyz="0 0 0" rpy="0 1.57 1.57"/>
+      <geometry>
+        <mesh filename="package://seed_r7_description/meshes/typeF_upperbody/wrist.dae" scale="1 1 1" />
+      </geometry>
+    </collision> </xacro:unless>
+    <inertial>
+      <mass value="0.05" />
+      <origin xyz="0 0 0" rpy="0 -0 0"/>
+      <inertia ixx="0.0001" ixy="0" ixz="0" iyy="0.0001" iyz="0" izz="0.0001"/>
+    </inertial>
+  </link>
   <joint name="waist_y_joint" type="revolute">
     <parent link="${base_link}"/>
@@ -468,5 +506,5 @@
   <joint name="l_wrist_r_joint" type="revolute">
     <parent link="l_wrist_center"/>
-    <child  link="${l_hand_link}"/>
+    <child  link="l_wrist_top"/>
     <origin xyz="0 0 0" rpy="0 -0 0 "/>
     <axis   xyz="1 0 0"/>
@@ -475,5 +513,4 @@
     <dynamics damping="0.2" friction="0" />
   </joint>
-  <xacro:gazebo_transmission joint_name="l_wrist_r_joint" />
   <joint name="neck_y_joint" type="revolute">
     <parent link="body_link"/>
@@ -568,5 +605,5 @@
   <joint name="r_wrist_r_joint" type="revolute">
     <parent link="r_wrist_center"/>
-    <child  link="${r_hand_link}"/>
+    <child  link="r_wrist_top"/>
     <origin xyz="0 0 0" rpy="0 -0 0 "/>
     <axis   xyz="1 0 0"/>
