Commit message: added collision model of hand

File: seed_r7_description/typefcety/noid-upper.urdf.xacro (robot description, xacro)
@@ -14,10 +14,10 @@
     <parent link="r_hand_yaw_link"/>
     <child link="r_hand_link"/>
-    <origin xyz="0.0 0.0 -0.02" rpy="0 0 0 "/>
+    <origin xyz="0.0 0.0 -0.01" rpy="0 0 0 "/>
   </joint>
   <joint name="l_hand_connector" type="fixed">
     <parent link="l_hand_yaw_link"/>
     <child link="l_hand_link"/>
-    <origin xyz="0.0 0.0 -0.02" rpy="0 0 0 "/>
+    <origin xyz="0.0 0.0 -0.01" rpy="0 0 0 "/>
   </joint>
   <joint name="upper_lower_connector" type="fixed">

File: seed_r7_description/urdf/hand_yaw/hand_yaw.urdf.xacro (robot description, xacro)
@@ -10,9 +10,17 @@
   <link name="${prefix}_hand_yaw_link">
     <xacro:unless value="${disable_mesh}"> <visual>
-      <origin xyz="0.0 0 0.0" rpy="0 3.14 3.14"/>
+      <origin xyz="0.0 0 0.0" rpy="0 ${M_PI} ${M_PI}"/>
       <geometry>
         <mesh filename="package://seed_r7_description/meshes/hand_yaw/hand_yaw.dae" scale="1 1 1" />
       </geometry>
     </visual> </xacro:unless>
+    <xacro:unless value="${disable_mesh}">
+    <collision>
+      <origin xyz="0 0 -0.005" rpy="0 ${M_PI} ${M_PI}" />
+      <geometry>
+        <cylinder length="0.01" radius="0.03" />
+      </geometry>
+    </collision>
+    </xacro:unless>
     <inertial>
       <mass value="0.183" />

File: seed_r7_description/urdf/trx_s/trx_s.urdf.xacro (robot description, xacro)
@@ -11,4 +11,23 @@
       <origin xyz="0 0 0" rpy="${M_PI} 0 ${reflect * M_PI / 2.0}"/>
     </visual>
+    <xacro:unless value="${disable_mesh}">
+    <collision>
+     <origin rpy="${reflect * 0.7} 0 0" xyz="0 0 -0.075"/>
+     <geometry>
+       <box size="0.036 0.070 0.030" />
+     </geometry>
+    </collision>
+    <collision>
+     <origin rpy="0 0 0" xyz="0 0 -0.036"/>
+     <geometry>
+      <box size="0.036 0.050 0.070" />
+     </geometry>
+    </collision>
+    </xacro:unless>
+    <inertial>
+      <mass value="0.183" />
+      <origin xyz="0 0 -0.0875" rpy="0 0 0" />
+      <inertia ixx="0.000601" ixy="0" ixz="0" iyy="0.00055" iyz="0" izz="0.000102" />
+    </inertial>
   </link>
 <!-- hand index base -->
@@ -20,9 +39,22 @@
       <origin xyz="0 0 0" rpy="${M_PI} 0 ${reflect * M_PI / 2.0}"/>
     </visual>
+    <xacro:unless value="${disable_mesh}">
+    <collision>
+     <origin xyz="0 0 -0.02141" rpy="${M_PI / 2.0} 0 0"/>
+     <geometry>
+      <box size="0.041 0.061 0.010" />
+     </geometry>
+    </collision>
+    </xacro:unless>
+    <inertial>
+      <mass value="0.1" />
+      <origin xyz="0 ${reflect * 0.014} -0.021" rpy="0 0 0" />
+      <inertia ixx="0.001" ixy="0" ixz="0" iyy="0.0001" iyz="0" izz="0.0001" />
+    </inertial>
   </link>
   <joint name="${prefix}_indexbase_joint" type="continuous">
     <parent link="${prefix}_hand_link"/>
     <child  link="${prefix}_indexbase_link"/>
-    <origin xyz="0 ${-0.013*reflect} -0.087" rpy="0 0 0"/>
+    <origin xyz="0 ${-0.013*reflect} -0.087" rpy="${reflect * -0.3} 0 0"/>
     <axis   xyz="1 0 0"/>
     <limit lower="-3.14159" upper="3.14159" effort="25" velocity="0.5" />
@@ -36,4 +68,17 @@
       <origin xyz="0 0 0" rpy="${M_PI} 0 ${reflect * M_PI / 2.0}"/>
     </visual>
+    <xacro:unless value="${disable_mesh}">
+    <collision>
+      <origin xyz="0 0 -0.008" rpy="${M_PI / 2.0} 0 0"/>
+      <geometry>
+        <box size="0.034 0.030 0.010" />
+      </geometry>
+    </collision>
+    </xacro:unless>
+    <inertial>
+      <mass value="0.1" />
+      <origin xyz="0 ${reflect * 0.014} -0.008" rpy="0 0 0" />
+      <inertia ixx="0.001" ixy="0" ixz="0" iyy="0.0001" iyz="0" izz="0.0001" />
+    </inertial>
   </link>
   <joint name="${prefix}_indexmid_joint" type="continuous">
@@ -52,4 +97,17 @@
       <origin xyz="0 0 0" rpy="${M_PI} 0 ${reflect * M_PI / 2.0}"/>
     </visual>
+  <xacro:unless value="${disable_mesh}">
+  <collision>
+    <origin xyz="0 ${reflect * 0.013} 0.004" rpy="0 0 0"/>
+    <geometry>
+      <box size="0.040 0.028 0.016" />
+    </geometry>
+  </collision>
+  </xacro:unless>
+  <inertial>
+      <mass value="0.1" />
+      <origin xyz="0 ${reflect * 0.02} 0" rpy="0 0 0" />
+      <inertia ixx="0.0001" ixy="0" ixz="0" iyy="0.0001" iyz="0" izz="0.0001" />
+    </inertial>
   </link>
   <joint name="${prefix}_indexend_joint" type="continuous">
@@ -68,4 +126,23 @@
       <origin xyz="0 0 0" rpy="${M_PI} 0 ${reflect * M_PI / 2.0}"/>
     </visual>
+    <xacro:unless value="${disable_mesh}">
+    <collision>
+      <origin xyz="0.0 ${reflect * 0.019645} 0.01" rpy="${reflect * -1.6} 0 0" />
+      <geometry>
+        <box size="0.012 0.008 0.050" />
+      </geometry>
+    </collision>
+    <collision>
+      <origin xyz="0.0 ${reflect * 0.057} 0.0" rpy="${reflect * -2.0} 0 0" />
+      <geometry>
+        <box size="0.012 0.008 0.050" />
+      </geometry>
+    </collision>
+    </xacro:unless>
+    <inertial>
+      <mass value="0.1" />
+      <origin xyz="0 ${reflect * 0.05} -0.06" rpy="0 0 0" />
+      <inertia ixx="0.001" ixy="0" ixz="0" iyy="0.0001" iyz="0" izz="0.0001" />
+    </inertial>
   </link>
   <joint name="${prefix}_thumb_joint" type="revolute">
