Commit message: modify elbow joint of typeG to use mimic joint

File: seed_r7_description/typeg/noid.urdf (robot description, URDF)
Before this commit: robot SEED-Noid-Mover-typeG, 63 links, 62 joints
Links:
- removed link camera_frame
- removed link camera_optical_frame
- added link chest_camera_depth_optical_frame
- added link chest_camera_link
- added link chest_camera_right_ir_frame
- added link front_camera_depth_optical_frame
- added link l_elbow_middle_link, mass 0.162; collision mesh filename=package://seed_r7_description/meshes/typeG_upperbody/elbow_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 scale=1 1 1; visual mesh filename=package://seed_r7_description/meshes/typeG_upperbody/elbow_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 scale=1 1 1
- added link l_elbow_virtual_link, mass 0.001
- added link l_elbow_virtual_link_dummy, mass 0.001
- added link r_elbow_middle_link, mass 0.162; collision mesh filename=package://seed_r7_description/meshes/typeG_upperbody/elbow_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 scale=1 1 1; visual mesh filename=package://seed_r7_description/meshes/typeG_upperbody/elbow_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 scale=1 1 1
- added link r_elbow_virtual_link, mass 0.001
- added link r_elbow_virtual_link_dummy, mass 0.001
- added link rear_camera_depth_optical_frame
- link hip_center: geometry collision sphere radius=0.05; visual mesh filename=package://seed_r7_description/meshes/typeG_upperbody/hip_ce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 scale=1 1 1
- link hip_sphere_link: geometry collision sphere radius=0.05; visual mesh filename=package://seed_r7_description/meshes/typeG_upperbody/hip_sp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 scale=1 1 1
- link l_elbow_link: geometry collision mesh filename=package://seed_r7_description/meshes/typeG_upperbody/elbow_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 scale=1 1 1; visual mesh filename=package://seed_r7_description/meshes/typeG_upperbody/elbow_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 scale=1 1 1
- link l_upperarm_link: geometry collision mesh filename=package://seed_r7_description/meshes/typeG_upperbody/uppera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 scale=1 1 1; visual mesh filename=package://seed_r7_description/meshes/typeG_upperbody/uppera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 scale=1 1 1
- link r_elbow_link: geometry collision mesh filename=package://seed_r7_description/meshes/typeG_upperbody/elbow_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 scale=1 1 1; visual mesh filename=package://seed_r7_description/meshes/typeG_upperbody/elbow_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 scale=1 1 1
- link r_upperarm_link: geometry collision mesh filename=package://seed_r7_description/meshes/typeG_upperbody/uppera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 scale=1 1 1; visual mesh filename=package://seed_r7_description/meshes/typeG_upperbody/uppera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 scale=1 1 1
Joints:
- removed joint camera_optical
- removed joint camera_setting
- added joint body_link_to_chest_camera_link: type fixed, parent body_link, child chest_camera_link, origin xyz=0.058198 0.0 0.273087 rpy=0 0.698132 0
- added joint chest_camera_depth_optical_joint: type fixed, parent chest_camera_link, child chest_camera_depth_optical_frame, origin xyz=0 0 0 rpy=-1.57079632679 0 -1.57079632679
- added joint chest_camera_link_to_chest_camera_right_ir_link: type fixed, parent chest_camera_link, child chest_camera_right_ir_frame, origin xyz=0 -0.055 0 rpy=0 0 0
- added joint front_camera_depth_optical_joint: type fixed, parent front_camera_link, child front_camera_depth_optical_frame, origin xyz=0 0 0 rpy=-1.57079632679 0 -1.57079632679
- added joint l_elbow_joint_mimic: type continuous, parent l_elbow_virtual_link, child l_elbow_virtual_link_dummy, origin xyz=0.0 0 0 rpy=0 0 0 , axis 0 1 0, mimic joint=l_elbow_joint multiplier=-1 offset=0
- added joint l_elbow_middle_joint: type continuous, parent l_elbow_virtual_link_dummy, child l_elbow_middle_link, origin xyz=0.0 0 0 rpy=0 -0 0 , axis 0 1 0, mimic joint=l_elbow_joint multiplier=0.591222 offset=0
- added joint l_elbow_middle_joint_mimic: type continuous, parent l_elbow_middle_link, child l_elbow_link, origin xyz=0.0 0 -0.07 rpy=0 -0 0 , axis 0 1 0, mimic joint=l_elbow_joint multiplier=0.408778 offset=0
- added joint r_elbow_joint_mimic: type continuous, parent r_elbow_virtual_link, child r_elbow_virtual_link_dummy, origin xyz=0.0 0 0 rpy=0 0 0 , axis 0 1 0, mimic joint=r_elbow_joint multiplier=-1 offset=0
- added joint r_elbow_middle_joint: type continuous, parent r_elbow_virtual_link_dummy, child r_elbow_middle_link, origin xyz=0.0 0 0 rpy=0 -0 0 , axis 0 1 0, mimic joint=r_elbow_joint multiplier=0.591222 offset=0
- added joint r_elbow_middle_joint_mimic: type continuous, parent r_elbow_middle_link, child r_elbow_link, origin xyz=0.0 0 -0.07 rpy=0 -0 0 , axis 0 1 0, mimic joint=r_elbow_joint multiplier=0.408778 offset=0
- added joint rear_camera_depth_optical_joint: type fixed, parent rear_camera_link, child rear_camera_depth_optical_frame, origin xyz=0 0 0 rpy=-1.57079632679 0 -1.57079632679
- joint l_elbow_joint: child l_elbow_link -> l_elbow_virtual_link; limit lower=-2.96 upper=0 effort=100 velocity=4.4 -> lower=-3.0 upper=0 effort=100 velocity=1.1; origin xyz=0.02803 0 -0.229460 rpy=0 -0 0  -> xyz=0.0 0 -0.2085 rpy=0 -0 0 
- joint l_shoulder_p_joint: limit lower=-1.55 upper=0.29 effort=200 velocity=0.6 -> lower=-1.55 upper=0.29 effort=200 velocity=0.4
- joint l_shoulder_r_joint: limit lower=-0.08 upper=1.57 effort=100 velocity=1.0 -> lower=-0.08 upper=1.57 effort=100 velocity=0.5
- joint l_shoulder_y_joint: limit lower=-1.57 upper=1.57 effort=100 velocity=1.7 -> lower=-1.57 upper=1.57 effort=100 velocity=1.1
- joint l_wrist_p_joint: limit lower=-0.12 upper=0.12 effort=100 velocity=1.7 -> lower=-0.12 upper=0.12 effort=100 velocity=0.8
- joint l_wrist_r_joint: limit lower=-1.57 upper=0.34 effort=100 velocity=3.4 -> lower=-1.57 upper=0.34 effort=100 velocity=1.8
- joint l_wrist_y_joint: limit lower=-1.57 upper=1.57 effort=100 velocity=1.9 -> lower=-1.57 upper=1.57 effort=100 velocity=1.2; origin xyz=-0.02096 0 -0.137530 rpy=0 -0 0  -> xyz=0.0 0 -0.1095 rpy=0 -0 0 
- joint neck_p_joint: limit lower=-0.34 upper=0.52 effort=100 velocity=4.0 -> lower=-0.34 upper=0.52 effort=100 velocity=2.1
- joint neck_r_joint: limit lower=-0.34 upper=0.34 effort=100 velocity=1.6 -> lower=-0.34 upper=0.34 effort=100 velocity=0.8
- joint r_elbow_joint: child r_elbow_link -> r_elbow_virtual_link; limit lower=-2.96 upper=0 effort=100 velocity=4.4 -> lower=-3.0 upper=0 effort=100 velocity=1.1; origin xyz=0.02803 0 -0.229460 rpy=0 -0 0  -> xyz=0.0 0 -0.2085 rpy=0 -0 0 
- joint r_shoulder_p_joint: limit lower=-1.55 upper=0.29 effort=200 velocity=0.6 -> lower=-1.55 upper=0.29 effort=200 velocity=0.4
- joint r_shoulder_r_joint: limit lower=-1.57 upper=0.08 effort=100 velocity=1.0 -> lower=-1.57 upper=0.08 effort=100 velocity=0.5
- joint r_shoulder_y_joint: limit lower=-1.57 upper=1.57 effort=100 velocity=1.7 -> lower=-1.57 upper=1.57 effort=100 velocity=1.1
- joint r_wrist_p_joint: limit lower=-0.12 upper=0.12 effort=100 velocity=1.7 -> lower=-0.12 upper=0.12 effort=100 velocity=0.8
- joint r_wrist_r_joint: limit lower=-0.34 upper=1.57 effort=100 velocity=3.4 -> lower=-0.34 upper=1.57 effort=100 velocity=1.8
- joint r_wrist_y_joint: limit lower=-1.57 upper=1.57 effort=100 velocity=1.9 -> lower=-1.57 upper=1.57 effort=100 velocity=1.2; origin xyz=-0.02096 0 -0.137530 rpy=0 -0 0  -> xyz=0.0 0 -0.1095 rpy=0 -0 0 
- joint waist_p_joint: limit lower=-0.17 upper=0.69 effort=2000 velocity=1.6 -> lower=-0.17 upper=0.69 effort=500 velocity=0.4
- joint waist_r_joint: limit lower=-0.12 upper=0.12 effort=2000 velocity=1.3 -> lower=-0.12 upper=0.12 effort=500 velocity=0.3
- joint waist_y_joint: limit lower=-2.09 upper=2.09 effort=500 velocity=1.7 -> lower=-2.09 upper=2.09 effort=500 velocity=0.6
- joint wheel_base_link_to_front_camera_base_link: origin xyz=0.31815 0 0.0165 rpy=0 0 0 -> xyz=0.31815 0 0.0185 rpy=0 0 0
- joint wheel_base_link_to_rear_camera_base_link: origin xyz=-0.31815 0 0.0165 rpy=0 0 3.1415926538 -> xyz=-0.31815 0 0.0185 rpy=0 0 3.1415926538
- joint wheels_body_to_base_laser_connector: origin xyz=0.308 0 0.0994 rpy=0 0 0 -> xyz=0.308 0 0.1014 rpy=0 0 0

File: seed_r7_description/typeg/noid.urdf.xacro (robot description, xacro)
@@ -11,4 +11,5 @@
  <!-- gazebo settings -->
  <!-- camera -->
+ <!--
  <link name="camera_frame" />
  <link name="camera_optical_frame" />
@@ -23,6 +24,39 @@
    <origin xyz="0 0 0" rpy="-1.570796326795 0 -1.570796326795" />
  </joint>
+ -->
+<!--
  <xacro:gazebo_camera link_name="camera_frame"
                       frame_name="camera_optical_frame" />
+-->
+<xacro:property  name="camera_name" value="front_camera"/>
+<link name="${camera_name}_depth_optical_frame"/>
+<joint name="${camera_name}_depth_optical_joint" type="fixed">
+  <origin xyz="0 0 0" rpy="${-M_PI/2} 0 ${-M_PI/2}" />
+  <parent link="${camera_name}_link" />
+  <child link="${camera_name}_depth_optical_frame" />
+</joint>
+<xacro:gazebo_depth_camera link_name="${camera_name}_link"
+                      frame_name="${camera_name}_depth_optical_frame"
+                      camera_name="${camera_name}"/>
+<xacro:property  name="camera_name" value="rear_camera"/>
+<link name="${camera_name}_depth_optical_frame"/>
+<joint name="${camera_name}_depth_optical_joint" type="fixed">
+  <origin xyz="0 0 0" rpy="${-M_PI/2} 0 ${-M_PI/2}" />
+  <parent link="${camera_name}_link" />
+  <child link="${camera_name}_depth_optical_frame" />
+</joint>
+<xacro:gazebo_depth_camera link_name="${camera_name}_link"
+                      frame_name="${camera_name}_depth_optical_frame"
+                      camera_name="${camera_name}"/>
+<xacro:property  name="camera_name" value="chest_camera"/>
+<link name="${camera_name}_depth_optical_frame"/>
+<joint name="${camera_name}_depth_optical_joint" type="fixed">
+  <origin xyz="0 0 0" rpy="${-M_PI/2} 0 ${-M_PI/2}" />
+  <parent link="${camera_name}_link" />
+  <child link="${camera_name}_depth_optical_frame" />
+</joint>
+<xacro:gazebo_depth_camera link_name="${camera_name}_link"
+                      frame_name="${camera_name}_depth_optical_frame"
+                      camera_name="${camera_name}"/>
  <!-- laser -->
  <xacro:gazebo_laser_sensor link_name="wheels_base_laser_link"
@@ -37,63 +71,23 @@
      <!-- lifter -->
      <mimic joint="knee_joint"  offset="0.0" multiplier="-1.0"
-            P="4000" I="0.1" D="80" i_max="500" i_min="-500"
-            command_max="2000" command_min="-2000">
+            P="100" I="0.1" D="10" i_max="500" i_min="-500"
+            command_max="2000" command_min="-2000" velocity='true'>
        knee_joint_mimic
-       <joint> knee_joint </joint>
-       <offset> 0.0 </offset>
-       <multiplier> -1.0 </multiplier>
-       <P> 4000 </P>
-       <I> 0.1 </I>
-       <D> 80 </D>
-       <i_max>  500 </i_max>
-       <i_min> -500 </i_min>
-       <command_max>  2000 </command_max>
-       <command_min> -2000 </command_min>
      </mimic>
      <mimic joint="ankle_joint"  offset="0.0" multiplier="-1.0"
-            P="4000" I="0.1" D="80" i_max="500" i_min="-500"
-            command_max="2000" command_min="-2000">
+            P="100" I="0.1" D="10" i_max="500" i_min="-500"
+            command_max="2000" command_min="-2000" velocity='true'>
        ankle_joint_mimic
-       <joint> ankle_joint </joint>
-       <offset> 0.0 </offset>
-       <multiplier> -1.0 </multiplier>
-       <P> 4000 </P>
-       <I> 0.1 </I>
-       <D> 80 </D>
-       <i_max>  500 </i_max>
-       <i_min> -500 </i_min>
-       <command_max>  2000 </command_max>
-       <command_min> -2000 </command_min>
      </mimic>
      <!-- lifter(dummy) -->
      <mimic joint="knee_joint"  offset="0.0" multiplier="-1.0"
-            P="1000" I="0.0" D="1" i_max="0" i_min="0"
-            command_max="200" command_min="-200">
+            P="100" I="0.0" D="10" i_max="0" i_min="0"
+            command_max="200" command_min="-200" velocity='true'>
        knee_joint_dummy
-       <joint> knee_joint </joint>
-       <offset> 0.0 </offset>
-       <multiplier> -1.0 </multiplier>
-       <P> 1000 </P>
-       <I> 0.0 </I>
-       <D> 1 </D>
-       <i_max>  0 </i_max>
-       <i_min> -0 </i_min>
-       <command_max>  200 </command_max>
-       <command_min> -200 </command_min>
      </mimic>
      <mimic joint="ankle_joint"  offset="0.0" multiplier="1.0"
-            P="1000" I="0.0" D="1" i_max="0" i_min="0"
-            command_max="200" command_min="-200">
+            P="100" I="0.0" D="10" i_max="0" i_min="0"
+            command_max="200" command_min="-200"  velocity='true'>
        ankle_joint_dummy
-       <joint> ankle_joint </joint>
-       <offset> 0.0 </offset>
-       <multiplier> 1.0 </multiplier>
-       <P> 1000 </P>
-       <I> 0.0 </I>
-       <D> 1 </D>
-       <i_max>  0 </i_max>
-       <i_min> -0 </i_min>
-       <command_max>  200 </command_max>
-       <command_min> -200 </command_min>
      </mimic>
      <!-- lhand -->
@@ -102,14 +96,4 @@
             command_max="50" command_min="-50">
        l_indexbase_joint
-       <joint> l_thumb_joint </joint>
-       <offset> 0.0 </offset>
-       <multiplier> -1.0 </multiplier>
-       <P> 30 </P>
-       <I> 0.0 </I>
-       <D> 0.03 </D>
-       <i_max>  0 </i_max>
-       <i_min> -0 </i_min>
-       <command_max>  50 </command_max>
-       <command_min> -50 </command_min>
      </mimic>
      <mimic joint="l_thumb_joint"  offset="-0.2" multiplier="-0.3"
@@ -117,14 +101,4 @@
             command_max="50" command_min="-50">
        l_indexmid_joint
-       <joint> l_thumb_joint </joint>
-       <offset> -0.2 </offset>
-       <multiplier> -0.3 </multiplier>
-       <P> 30 </P>
-       <I> 0.0 </I>
-       <D> 0.03 </D>
-       <i_max>  0 </i_max>
-       <i_min> -0 </i_min>
-       <command_max>  50 </command_max>
-       <command_min> -50 </command_min>
      </mimic>
      <mimic joint="l_thumb_joint"  offset="-0.2" multiplier="-0.3"
@@ -132,14 +106,4 @@
             command_max="50" command_min="-50">
        l_indexend_joint
-       <joint> l_thumb_joint </joint>
-       <offset> -0.2 </offset>
-       <multiplier> -0.3 </multiplier>
-       <P> 30 </P>
-       <I> 0.0 </I>
-       <D> 0.03 </D>
-       <i_max>  0 </i_max>
-       <i_min> -0 </i_min>
-       <command_max>  50 </command_max>
-       <command_min> -50 </command_min>
      </mimic>
      <!-- rhand -->
@@ -148,14 +112,4 @@
             command_max="50" command_min="-50">
        r_indexbase_joint
-       <joint> r_thumb_joint </joint>
-       <offset> 0.0 </offset>
-       <multiplier> -1.0 </multiplier>
-       <P> 30 </P>
-       <I> 0.0 </I>
-       <D> 0.03 </D>
-       <i_max>  0 </i_max>
-       <i_min> -0 </i_min>
-       <command_max>  50 </command_max>
-       <command_min> -50 </command_min>
      </mimic>
      <mimic joint="r_thumb_joint"  offset="0.2" multiplier="-0.3"
@@ -163,14 +117,4 @@
             command_max="50" command_min="-50">
        r_indexmid_joint
-       <joint> r_thumb_joint </joint>
-       <offset> 0.2 </offset>
-       <multiplier> -0.3 </multiplier>
-       <P> 30 </P>
-       <I> 0.0 </I>
-       <D> 0.03 </D>
-       <i_max>  0 </i_max>
-       <i_min> -0 </i_min>
-       <command_max>  50 </command_max>
-       <command_min> -50 </command_min>
      </mimic>
      <mimic joint="r_thumb_joint"  offset="0.2" multiplier="-0.3"
@@ -178,14 +122,36 @@
             command_max="50" command_min="-50">
        r_indexend_joint
-       <joint> r_thumb_joint </joint>
-       <offset> 0.2 </offset>
-       <multiplier> -0.3 </multiplier>
-       <P> 30 </P>
-       <I> 0.0 </I>
-       <D> 0.03 </D>
-       <i_max>  0 </i_max>
-       <i_min> -0 </i_min>
-       <command_max>  50 </command_max>
-       <command_min> -50 </command_min>
+     </mimic>
+      <!-- r_elbow -->
+     <mimic joint="r_elbow_joint"  offset="0.0" multiplier="-1.0"
+            P="100" I="0.01" D="10" i_max="0" i_min="-0"
+            command_max="50" command_min="-50" velocity='true'>
+       r_elbow_joint_mimic
+     </mimic>
+     <mimic joint="r_elbow_joint"  offset="0.0" multiplier="0.591"
+            P="100" I="0.01" D="10" i_max="0" i_min="-0"
+            command_max="50" command_min="-50" velocity='true'>
+       r_elbow_middle_joint
+     </mimic>
+     <mimic joint="r_elbow_joint"  offset="0.0" multiplier="0.409"
+            P="100" I="0.01" D="10" i_max="0" i_min="-0"
+            command_max="50" command_min="-50" velocity='true'>
+       r_elbow_middle_joint_mimic
+     </mimic>
+     <!-- l_elbow -->
+     <mimic joint="l_elbow_joint"  offset="0.0" multiplier="-1.0"
+            P="100" I="0.01" D="10" i_max="0" i_min="-0"
+            command_max="50" command_min="-50" velocity='true'>
+       l_elbow_joint_mimic
+     </mimic>
+     <mimic joint="l_elbow_joint"  offset="0.0" multiplier="0.591"
+            P="100" I="0.01" D="10" i_max="0" i_min="-0"
+            command_max="50" command_min="-50" velocity='true'>
+       l_elbow_middle_joint
+     </mimic>
+     <mimic joint="l_elbow_joint"  offset="0.0" multiplier="0.409"
+            P="100" I="0.01" D="10" i_max="0" i_min="-0"
+            command_max="50" command_min="-50" velocity='true'>
+       l_elbow_middle_joint_mimic
      </mimic>
    </plugin>

File: seed_r7_description/urdf/gazebo.xacro (robot description, xacro)
@@ -17,13 +17,13 @@
       <joint name="${joint_name}">
         <!-- dupricated in kinetic -->
-        <!--hardwareInterface>hardware_interface/EffortJointInterface</hardwareInterface-->
-        <!--hardwareInterface>EffortJointInterface</hardwareInterface-->
-        <hardwareInterface>VelocityJointInterface</hardwareInterface>
+        <!-- <hardwareInterface>hardware_interface/PositionJointInterface</hardwareInterface> -->
+        <!--<hardwareInterface>hardware_interface/EffortJointInterface</hardwareInterface>-->
+        <hardwareInterface>hardware_interface/VelocityJointInterface</hardwareInterface>
       </joint>
       <actuator name="${joint_name}_motor">
         <!-- dupricated in kinetic -->
-        <!--hardwareInterface>hardware_interface/EffortJointInterface</hardwareInterface-->
-        <!--hardwareInterface>EffortJointInterface</hardwareInterface-->
-        <hardwareInterface>VelocityJointInterface</hardwareInterface>
+        <!-- <hardwareInterface>hardware_interface/PositionJointInterface</hardwareInterface> -->
+        <!--<hardwareInterface>hardware_interface/EffortJointInterface</hardwareInterface>-->
+        <hardwareInterface>hardware_interface/VelocityJointInterface</hardwareInterface>
         <mechanicalReduction>1</mechanicalReduction>
       </actuator>
@@ -36,4 +36,5 @@
         <robotNamespace>${namespace}</robotNamespace>
         <robotSimType>gazebo_ros_control/DefaultRobotHWSim</robotSimType>
+        <legacyModeNS>true</legacyModeNS>
       </plugin>
     </gazebo>

File: seed_r7_description/urdf/typeG_lifter/lifter.urdf.xacro (robot description, xacro)
@@ -98,5 +98,5 @@
       </visual>
       <collision>
-        <origin xyz="0 0 0.05" rpy="0 0 0"/>
+        <origin xyz="0 0 0" rpy="0 0 0"/>
         <geometry>
           <mesh filename="package://seed_r7_description/meshes/typeG_lifter/leg_base_link.dae" scale="1 1 1" />
@@ -131,4 +131,5 @@
       <axis xyz="0 -1 0"/>
       <limit effort="10000" lower="-1.5707" upper="0" velocity="0.5"/>
+      <dynamics damping="0.5" friction="0.1" />
     </joint>
     <xacro:gazebo_transmission joint_name="knee_joint" />
@@ -139,5 +140,5 @@
       <axis   xyz="0 -1 0"/>
       <limit effort="10000" lower="0" upper="1.5707" velocity="0.5" />
-      <dynamics damping="0.2" friction="0" />
+      <dynamics damping="0.5" friction="0.1" />
     </joint>
     <xacro:gazebo_transmission joint_name="ankle_joint" />
