Commit message: modify elbow joint of typeG to use mimic joint

File: seed_r7_description/urdf/typeG_upperbody/noid_upper_typeg.urdf.xacro (robot description, xacro)
@@ -1,9 +1,9 @@
 <?xml version="1.0"?>
 <!-- XML namespaces -->
-<robot name="noid_upper_typef" xmlns:xacro="http://ros.org/wiki/xacro">
+<robot name="noid_upper_typeg" xmlns:xacro="http://ros.org/wiki/xacro">
   <xacro:include filename="$(find seed_r7_description)/urdf/gazebo.xacro" />
   <xacro:property name="wrist_sensor_offset" value="0.0"/>
   <xacro:macro name="noid_upper" params="base_link disable_mesh:=false r_hand_link:=r_hand_link l_hand_link:=l_hand_link">
-  <!-- ============================   typeF_upper   ============================ -->
+  <!-- ============================   typeG_upper   ============================ -->
   <link name="${base_link}">
     <xacro:unless value="${disable_mesh}"> <visual>
@@ -34,7 +34,8 @@
     </visual> </xacro:unless>
     <xacro:unless value="${disable_mesh}"> <collision>
-      <origin xyz="0 0 0" rpy="0 0 0"/>
-      <geometry>
-        <mesh filename="package://seed_r7_description/meshes/typeG_upperbody/hip_sphere_link.dae" scale="1 1 1" />
+      <origin xyz="0 0 0.132" rpy="0 0 0"/>
+      <geometry>
+        <!-- <mesh filename="package://seed_r7_description/meshes/typeG_upperbody/hip_sphere_link.dae" scale="1 1 1" /> -->
+        <sphere radius="0.05"/>
       </geometry>
     </collision> </xacro:unless>
@@ -58,5 +59,6 @@
       <origin xyz="0 0 0" rpy="0 0 0"/>
       <geometry>
-        <mesh filename="package://seed_r7_description/meshes/typeG_upperbody/hip_center_link.dae" scale="1 1 1" />
+        <!-- <mesh filename="package://seed_r7_description/meshes/typeG_upperbody/hip_center_link.dae" scale="1 1 1" /> -->
+        <sphere radius="0.05"/>
       </geometry>
     </collision> </xacro:unless>
@@ -136,11 +138,11 @@
       <origin xyz="0 0 0" rpy="0 -0 0"/>
       <geometry>
-        <mesh filename="package://seed_r7_description/meshes/typeG_upperbody/l_upperarm_link.dae" scale="1 1 1" />
-      </geometry>
-    </visual> </xacro:unless>
-    <xacro:unless value="${disable_mesh}"> <collision>
-      <origin xyz="0 0 0" rpy="0 -0 0"/>
-      <geometry>
-        <mesh filename="package://seed_r7_description/meshes/typeG_upperbody/l_upperarm_link.dae" scale="1 1 1" />
+        <mesh filename="package://seed_r7_description/meshes/typeG_upperbody/upperarm_link.dae" scale="1 1 1" />
+      </geometry>
+    </visual> </xacro:unless>
+    <xacro:unless value="${disable_mesh}"> <collision>
+      <origin xyz="0 0 0" rpy="0 -0 0"/>
+      <geometry>
+        <mesh filename="package://seed_r7_description/meshes/typeG_upperbody/upperarm_link.dae" scale="1 1 1" />
       </geometry>
     </collision> </xacro:unless>
@@ -155,15 +157,51 @@
   </link>
   <xacro:gazebo_link_reference link_name="l_upperarm_link" />
+  <link name="l_elbow_virtual_link">
+    <inertial>
+      <mass value="0.001" />
+      <origin xyz="0 0 0" rpy="0 0 0"/>
+      <inertia ixx="0.01" ixy="0" ixz="0" iyy="0.01" iyz="0" izz="0.01"/>
+    </inertial>
+  </link>
+  <xacro:gazebo_link_reference link_name="l_elbow_virtual_link" />
+  <link name="l_elbow_virtual_link_dummy">
+    <inertial>
+      <mass value="0.001" />
+      <origin xyz="0 0 0" rpy="0 0 0"/>
+      <inertia ixx="0.01" ixy="0" ixz="0" iyy="0.01" iyz="0" izz="0.01"/>
+    </inertial>
+  </link>
+  <xacro:gazebo_link_reference link_name="l_elbow_virtual_link_dummy" />
+  <link name="l_elbow_middle_link">
+    <xacro:unless value="${disable_mesh}"> <visual>
+      <origin xyz="0 0 0" rpy="0 -0 0"/>
+      <geometry>
+        <mesh filename="package://seed_r7_description/meshes/typeG_upperbody/elbow_middle_link.dae" scale="1 1 1" />
+      </geometry>
+    </visual> </xacro:unless>
+    <xacro:unless value="${disable_mesh}"> <collision>
+      <origin xyz="0 0 0" rpy="0 -0 0"/>
+      <geometry>
+        <mesh filename="package://seed_r7_description/meshes/typeG_upperbody/elbow_middle_link.dae" scale="1 1 1" />
+      </geometry>
+    </collision> </xacro:unless>
+    <inertial>
+      <mass value="0.162" />
+      <origin xyz="-0.014 0 -0.032" rpy="0 -0 0"/>
+      <inertia ixx="0.00178" ixy="0" ixz="0" iyy="0.00179" iyz="0" izz="0.0035"/>
+    </inertial>
+  </link>
+  <xacro:gazebo_link_reference link_name="l_elbow_middle_link" />
   <link name="l_elbow_link">
     <xacro:unless value="${disable_mesh}"> <visual>
       <origin xyz="0 0 0" rpy="0 -0 0"/>
       <geometry>
-        <mesh filename="package://seed_r7_description/meshes/typeG_upperbody/l_elbow_link.dae" scale="1 1 1" />
-      </geometry>
-    </visual> </xacro:unless>
-    <xacro:unless value="${disable_mesh}"> <collision>
-      <origin xyz="0 0 0" rpy="0 -0 0"/>
-      <geometry>
-        <mesh filename="package://seed_r7_description/meshes/typeG_upperbody/l_elbow_link.dae" scale="1 1 1" />
+        <mesh filename="package://seed_r7_description/meshes/typeG_upperbody/elbow_link.dae" scale="1 1 1" />
+      </geometry>
+    </visual> </xacro:unless>
+    <xacro:unless value="${disable_mesh}"> <collision>
+      <origin xyz="0 0 0" rpy="0 -0 0"/>
+      <geometry>
+        <mesh filename="package://seed_r7_description/meshes/typeG_upperbody/elbow_link.dae" scale="1 1 1" />
       </geometry>
     </collision> </xacro:unless>
@@ -347,11 +385,11 @@
       <origin xyz="0 0 0" rpy="0 -0 0"/>
       <geometry>
-        <mesh filename="package://seed_r7_description/meshes/typeG_upperbody/r_upperarm_link.dae" scale="1 1 1" />
-      </geometry>
-    </visual> </xacro:unless>
-    <xacro:unless value="${disable_mesh}"> <collision>
-      <origin xyz="0 0 0" rpy="0 -0 0"/>
-      <geometry>
-        <mesh filename="package://seed_r7_description/meshes/typeG_upperbody/r_upperarm_link.dae" scale="1 1 1" />
+        <mesh filename="package://seed_r7_description/meshes/typeG_upperbody/upperarm_link.dae" scale="1 1 1" />
+      </geometry>
+    </visual> </xacro:unless>
+    <xacro:unless value="${disable_mesh}"> <collision>
+      <origin xyz="0 0 0" rpy="0 -0 0"/>
+      <geometry>
+        <mesh filename="package://seed_r7_description/meshes/typeG_upperbody/upperarm_link.dae" scale="1 1 1" />
       </geometry>
     </collision> </xacro:unless>
@@ -366,15 +404,51 @@
   </link>
   <xacro:gazebo_link_reference link_name="r_upperarm_link" />
+  <link name="r_elbow_virtual_link">
+    <inertial>
+      <mass value="0.001" />
+      <origin xyz="0 0 0" rpy="0 0 0"/>
+      <inertia ixx="0.01" ixy="0" ixz="0" iyy="0.01" iyz="0" izz="0.01"/>
+    </inertial>
+  </link>
+  <xacro:gazebo_link_reference link_name="r_elbow_virtual_link" />
+  <link name="r_elbow_virtual_link_dummy">
+    <inertial>
+      <mass value="0.001" />
+      <origin xyz="0 0 0" rpy="0 0 0"/>
+      <inertia ixx="0.01" ixy="0" ixz="0" iyy="0.01" iyz="0" izz="0.01"/>
+    </inertial>
+  </link>
+  <xacro:gazebo_link_reference link_name="r_elbow_virtual_link_dummy" />
+  <link name="r_elbow_middle_link">
+    <xacro:unless value="${disable_mesh}"> <visual>
+      <origin xyz="0 0 0" rpy="0 -0 0"/>
+      <geometry>
+        <mesh filename="package://seed_r7_description/meshes/typeG_upperbody/elbow_middle_link.dae" scale="1 1 1" />
+      </geometry>
+    </visual> </xacro:unless>
+    <xacro:unless value="${disable_mesh}"> <collision>
+      <origin xyz="0 0 0" rpy="0 -0 0"/>
+      <geometry>
+        <mesh filename="package://seed_r7_description/meshes/typeG_upperbody/elbow_middle_link.dae" scale="1 1 1" />
+      </geometry>
+    </collision> </xacro:unless>
+    <inertial>
+      <mass value="0.162" />
+      <origin xyz="-0.014 0 -0.032" rpy="0 -0 0"/>
+      <inertia ixx="0.00178" ixy="0" ixz="0" iyy="0.00179" iyz="0" izz="0.0035"/>
+    </inertial>
+  </link>
+  <xacro:gazebo_link_reference link_name="r_elbow_middle_link" />
   <link name="r_elbow_link">
     <xacro:unless value="${disable_mesh}"> <visual>
       <origin xyz="0 0 0" rpy="0 -0 0"/>
       <geometry>
-        <mesh filename="package://seed_r7_description/meshes/typeG_upperbody/r_elbow_link.dae" scale="1 1 1" />
-      </geometry>
-    </visual> </xacro:unless>
-    <xacro:unless value="${disable_mesh}"> <collision>
-      <origin xyz="0 0 0" rpy="0 -0 0"/>
-      <geometry>
-        <mesh filename="package://seed_r7_description/meshes/typeG_upperbody/r_elbow_link.dae" scale="1 1 1" />
+        <mesh filename="package://seed_r7_description/meshes/typeG_upperbody/elbow_link.dae" scale="1 1 1" />
+      </geometry>
+    </visual> </xacro:unless>
+    <xacro:unless value="${disable_mesh}"> <collision>
+      <origin xyz="0 0 0" rpy="0 -0 0"/>
+      <geometry>
+        <mesh filename="package://seed_r7_description/meshes/typeG_upperbody/elbow_link.dae" scale="1 1 1" />
       </geometry>
     </collision> </xacro:unless>
@@ -466,5 +540,5 @@
     <axis   xyz="0 1 0"/>
     <!-- from -10 to 40 degrees-->
-    <limit lower="-0.17" upper="0.69" effort="2000" velocity="0.4" />
+    <limit lower="-0.17" upper="0.69" effort="500" velocity="0.4" />
     <dynamics damping="0.2" friction="0" />
   </joint>
@@ -476,5 +550,5 @@
     <axis   xyz="1 0 0"/>
     <!-- from -7 to 7 degrees-->
-    <limit lower="-0.12" upper="0.12" effort="2000" velocity="0.3" />
+    <limit lower="-0.12" upper="0.12" effort="500" velocity="0.3" />
     <dynamics damping="0.2" friction="0" />
   </joint>
@@ -510,18 +584,8 @@
   </joint>
   <xacro:gazebo_transmission joint_name="l_shoulder_y_joint" />
-  <joint name="l_elbow_joint" type="revolute">
-    <parent link="l_upperarm_link"/>
-    <child  link="l_elbow_link"/>
-    <origin xyz="0.02803 0 -0.229460" rpy="0 -0 0 "/>
-    <axis   xyz="0 1 0"/>
-    <!-- from -170 to 0 degrees-->
-    <limit lower="-2.96" upper="0" effort="100" velocity="1.1" />
-    <dynamics damping="0.2" friction="0" />
-  </joint>
-  <xacro:gazebo_transmission joint_name="l_elbow_joint" />
   <joint name="l_wrist_y_joint" type="revolute">
     <parent link="l_elbow_link"/>
     <child  link="l_forearm_link"/>
-    <origin xyz="-0.02096 0 -0.137530" rpy="0 -0 0 "/>
+    <origin xyz="0.0 0 -0.1095" rpy="0 -0 0 "/>
     <axis   xyz="0 0 1"/>
     <!-- from -90 to 90 degrees-->
@@ -549,5 +613,5 @@
     <dynamics damping="0.2" friction="0" />
   </joint>
-  <xacro:gazebo_transmission joint_name="r_wrist_r_joint" />
+  <xacro:gazebo_transmission joint_name="l_wrist_r_joint" />
   <joint name="l_wrist_to_hand_connector" type="fixed">
     <parent link="l_wrist_r_link"/>
@@ -555,5 +619,5 @@
     <origin xyz="0 0 -0.003" rpy="0 0 0 "/>
   </joint>
-  <xacro:gazebo_transmission joint_name="r_wrist_r_joint" />
+  <!-- <xacro:gazebo_transmission joint_name="l_wrist_to_hand_connector" /> -->
   <joint name="neck_y_joint" type="revolute">
     <parent link="body_link"/>
@@ -617,18 +681,8 @@
   </joint>
   <xacro:gazebo_transmission joint_name="r_shoulder_y_joint" />
-  <joint name="r_elbow_joint" type="revolute">
-    <parent link="r_upperarm_link"/>
-    <child  link="r_elbow_link"/>
-    <origin xyz="0.02803 0 -0.229460" rpy="0 -0 0 "/>
-    <axis   xyz="0 1 0"/>
-    <!-- from -170 to 0 degrees-->
-    <limit lower="-2.96" upper="0" effort="100" velocity="1.1" />
-    <dynamics damping="0.2" friction="0" />
-  </joint>
-  <xacro:gazebo_transmission joint_name="r_elbow_joint" />
   <joint name="r_wrist_y_joint" type="revolute">
     <parent link="r_elbow_link"/>
     <child  link="r_forearm_link"/>
-    <origin xyz="-0.02096 0 -0.137530" rpy="0 -0 0 "/>
+    <origin xyz="0.0 0 -0.1095" rpy="0 -0 0 "/>
     <axis   xyz="0 0 1"/>
     <!-- from -90 to 90 degrees-->
@@ -662,5 +716,79 @@
     <origin xyz="0 0 -0.003" rpy="0 0 0 "/>
   </joint>
-  <xacro:gazebo_transmission joint_name="r_wrist_r_joint" />
+  <!-- <xacro:gazebo_transmission joint_name="r_wrist_to_hand_connector" /> -->
+  <joint name="r_elbow_joint" type="revolute">
+    <parent link="r_upperarm_link"/>
+    <child  link="r_elbow_virtual_link"/>
+    <origin xyz="0.0 0 -0.2085" rpy="0 -0 0 "/>
+    <axis   xyz="0 1 0"/>
+    <!-- from -170 to 0 degrees-->
+    <limit lower="-3.0" upper="0" effort="100" velocity="1.1" />
+    <dynamics damping="0.2" friction="0.1" />
+  </joint>
+  <xacro:gazebo_transmission joint_name="r_elbow_joint" />
+  <joint name="r_elbow_joint_mimic" type="continuous">
+    <parent link="r_elbow_virtual_link"/>
+    <child  link="r_elbow_virtual_link_dummy"/>
+    <origin xyz="0.0 0 0" rpy="0 0 0 "/>
+    <axis   xyz="0 1 0"/>
+    <mimic joint="r_elbow_joint" multiplier="-1" offset="0" />
+  </joint>
+  <joint name="r_elbow_middle_joint" type="continuous">
+    <parent link="r_elbow_virtual_link_dummy"/>
+    <child  link="r_elbow_middle_link"/>
+    <origin xyz="0.0 0 0" rpy="0 -0 0 "/>
+    <axis   xyz="0 1 0"/>
+    <mimic joint="r_elbow_joint" multiplier="0.591222" offset="0" />
+  </joint>
+  <joint name="r_elbow_middle_joint_mimic" type="continuous">
+    <parent link="r_elbow_middle_link"/>
+    <child  link="r_elbow_link"/>
+    <origin xyz="0.0 0 -0.07" rpy="0 -0 0 "/>
+    <axis   xyz="0 1 0"/>
+    <mimic joint="r_elbow_joint" multiplier="0.408778" offset="0" />
+  </joint>
+  <joint name="l_elbow_joint" type="revolute">
+    <parent link="l_upperarm_link"/>
+    <child  link="l_elbow_virtual_link"/>
+    <origin xyz="0.0 0 -0.2085" rpy="0 -0 0 "/>
+    <axis   xyz="0 1 0"/>
+    <!-- from -170 to 0 degrees-->
+    <limit lower="-3.0" upper="0" effort="100" velocity="1.1" />
+    <dynamics damping="0.2" friction="0.1" />
+  </joint>
+  <xacro:gazebo_transmission joint_name="l_elbow_joint" />
+  <joint name="l_elbow_joint_mimic" type="continuous">
+    <parent link="l_elbow_virtual_link"/>
+    <child  link="l_elbow_virtual_link_dummy"/>
+    <origin xyz="0.0 0 0" rpy="0 0 0 "/>
+    <axis   xyz="0 1 0"/>
+    <mimic joint="l_elbow_joint" multiplier="-1" offset="0" />
+  </joint>
+  <joint name="l_elbow_middle_joint" type="continuous">
+    <parent link="l_elbow_virtual_link_dummy"/>
+    <child  link="l_elbow_middle_link"/>
+    <origin xyz="0.0 0 0" rpy="0 -0 0 "/>
+    <axis   xyz="0 1 0"/>
+    <mimic joint="l_elbow_joint" multiplier="0.591222" offset="0" />
+  </joint>
+  <joint name="l_elbow_middle_joint_mimic" type="continuous">
+    <parent link="l_elbow_middle_link"/>
+    <child  link="l_elbow_link"/>
+    <origin xyz="0.0 0 -0.07" rpy="0 -0 0 "/>
+    <axis   xyz="0 1 0"/>
+    <mimic joint="l_elbow_joint" multiplier="0.408778" offset="0" />
+  </joint>
+  <link name="chest_camera_link"/>
+  <joint name="body_link_to_chest_camera_link" type="fixed">
+    <parent  link="body_link"/>
+    <child link="chest_camera_link"/>
+    <origin xyz="0.058198 0.0 0.273087" rpy="0 0.698132 0"/>
+  </joint>
+  <link name="chest_camera_right_ir_frame"/>
+  <joint name="chest_camera_link_to_chest_camera_right_ir_link" type="fixed">
+    <parent  link="chest_camera_link"/>
+    <child link="chest_camera_right_ir_frame"/>
+    <origin xyz="0 -0.055 0" rpy="0 0 0"/>  <!-- realsense d415-->
+  </joint>
   </xacro:macro>
 </robot>
