Commit message: change the elbow joint of typeF to mimic

File: seed_r7_description/typef/noid.urdf (robot description, URDF)
Before this commit: robot SEED-Noid-Mover-typeF, 61 links, 60 joints
Links:
- removed link camera_frame
- removed link camera_optical_frame
- added link chest_camera_depth_optical_frame
- added link chest_camera_link
- added link chest_camera_right_ir_frame
- added link front_camera_depth_optical_frame
- added link l_elbow_middle_link, mass 0.162; collision mesh filename=package://seed_r7_description/meshes/typeF_upperbody/elbow_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 scale=1 1 1; visual mesh filename=package://seed_r7_description/meshes/typeF_upperbody/elbow_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 scale=1 1 1
- added link l_elbow_virtual_link, mass 0.001
- added link l_elbow_virtual_link_dummy, mass 0.001
- added link r_elbow_middle_link, mass 0.162; collision mesh filename=package://seed_r7_description/meshes/typeF_upperbody/elbow_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 scale=1 1 1; visual mesh filename=package://seed_r7_description/meshes/typeF_upperbody/elbow_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 scale=1 1 1
- added link r_elbow_virtual_link, mass 0.001
- added link r_elbow_virtual_link_dummy, mass 0.001
- added link rear_camera_depth_optical_frame
Joints:
- removed joint camera_optical
- removed joint camera_setting
- added joint body_link_to_chest_camera_link: type fixed, parent body_link, child chest_camera_link, origin xyz=0.062143 0.0 0.322289  rpy=0 0.785398 0
- added joint chest_camera_depth_optical_joint: type fixed, parent chest_camera_link, child chest_camera_depth_optical_frame, origin xyz=0 0 0 rpy=-1.57079632679 0 -1.57079632679
- added joint chest_camera_link_to_chest_camera_right_ir_link: type fixed, parent chest_camera_link, child chest_camera_right_ir_frame, origin xyz=0 -0.055 0 rpy=0 0 0
- added joint front_camera_depth_optical_joint: type fixed, parent front_camera_link, child front_camera_depth_optical_frame, origin xyz=0 0 0 rpy=-1.57079632679 0 -1.57079632679
- added joint l_elbow_joint_mimic: type continuous, parent l_elbow_virtual_link, child l_elbow_virtual_link_dummy, origin xyz=0.0 0 0 rpy=0 0 0 , axis 0 1 0, mimic joint=l_elbow_joint multiplier=-1 offset=0
- added joint l_elbow_middle_joint: type continuous, parent l_elbow_virtual_link_dummy, child l_elbow_middle_link, origin xyz=0.0 0 0 rpy=0 -0 0 , axis 0 1 0, mimic joint=l_elbow_joint multiplier=0.591222 offset=0
- added joint l_elbow_middle_joint_mimic: type continuous, parent l_elbow_middle_link, child l_elbow_link, origin xyz=0.0 0 -0.07 rpy=0 -0 0 , axis 0 1 0, mimic joint=l_elbow_joint multiplier=0.408778 offset=0
- added joint r_elbow_joint_mimic: type continuous, parent r_elbow_virtual_link, child r_elbow_virtual_link_dummy, origin xyz=0.0 0 0 rpy=0 0 0 , axis 0 1 0, mimic joint=r_elbow_joint multiplier=-1 offset=0
- added joint r_elbow_middle_joint: type continuous, parent r_elbow_virtual_link_dummy, child r_elbow_middle_link, origin xyz=0.0 0 0 rpy=0 -0 0 , axis 0 1 0, mimic joint=r_elbow_joint multiplier=0.591222 offset=0
- added joint r_elbow_middle_joint_mimic: type continuous, parent r_elbow_middle_link, child r_elbow_link, origin xyz=0.0 0 -0.07 rpy=0 -0 0 , axis 0 1 0, mimic joint=r_elbow_joint multiplier=0.408778 offset=0
- added joint rear_camera_depth_optical_joint: type fixed, parent rear_camera_link, child rear_camera_depth_optical_frame, origin xyz=0 0 0 rpy=-1.57079632679 0 -1.57079632679
- joint l_elbow_joint: child l_elbow_link -> l_elbow_virtual_link; limit lower=-3.0 upper=0 effort=100 velocity=1.2 -> lower=-3.0 upper=0 effort=100 velocity=1.1; origin xyz=0.035 0 -0.1625 rpy=0 -0 0  -> xyz=0.0 0 -0.128 rpy=0 -0 0 
- joint l_wrist_y_joint: origin xyz=-0.035 0 -0.070 rpy=0 -0 0  -> xyz=0 0 -0.0355 rpy=0 -0 0 
- joint r_elbow_joint: child r_elbow_link -> r_elbow_virtual_link; limit lower=-3.0 upper=0 effort=100 velocity=1.2 -> lower=-3.0 upper=0 effort=100 velocity=1.1; origin xyz=0.035 0 -0.1625 rpy=0 -0 0  -> xyz=0.0 0 -0.128 rpy=0 -0 0 
- joint r_wrist_y_joint: origin xyz=-0.035 0 -0.070 rpy=0 -0 0  -> xyz=0 0 -0.0355 rpy=0 -0 0 

File: seed_r7_description/typef/noid.urdf.xacro (robot description, xacro)
@@ -11,4 +11,5 @@
  <!-- gazebo settings -->
  <!-- camera -->
+ <!--
  <link name="camera_frame" />
  <link name="camera_optical_frame" />
@@ -25,4 +26,35 @@
  <xacro:gazebo_camera link_name="camera_frame"
                       frame_name="camera_optical_frame" />
+ -->
+<xacro:property  name="camera_name" value="front_camera"/>
+<link name="${camera_name}_depth_optical_frame"/>
+<joint name="${camera_name}_depth_optical_joint" type="fixed">
+  <origin xyz="0 0 0" rpy="${-M_PI/2} 0 ${-M_PI/2}" />
+  <parent link="${camera_name}_link" />
+  <child link="${camera_name}_depth_optical_frame" />
+</joint>
+<xacro:gazebo_depth_camera link_name="${camera_name}_link"
+                      frame_name="${camera_name}_depth_optical_frame"
+                      camera_name="${camera_name}"/>
+<xacro:property  name="camera_name" value="rear_camera"/>
+<link name="${camera_name}_depth_optical_frame"/>
+<joint name="${camera_name}_depth_optical_joint" type="fixed">
+  <origin xyz="0 0 0" rpy="${-M_PI/2} 0 ${-M_PI/2}" />
+  <parent link="${camera_name}_link" />
+  <child link="${camera_name}_depth_optical_frame" />
+</joint>
+<xacro:gazebo_depth_camera link_name="${camera_name}_link"
+                      frame_name="${camera_name}_depth_optical_frame"
+                      camera_name="${camera_name}"/>
+<xacro:property  name="camera_name" value="chest_camera"/>
+<link name="${camera_name}_depth_optical_frame"/>
+<joint name="${camera_name}_depth_optical_joint" type="fixed">
+  <origin xyz="0 0 0" rpy="${-M_PI/2} 0 ${-M_PI/2}" />
+  <parent link="${camera_name}_link" />
+  <child link="${camera_name}_depth_optical_frame" />
+</joint>
+<xacro:gazebo_depth_camera link_name="${camera_name}_link"
+                      frame_name="${camera_name}_depth_optical_frame"
+                      camera_name="${camera_name}"/>
  <!-- laser -->
  <xacro:gazebo_laser_sensor link_name="wheels_base_laser_link"
@@ -37,63 +69,23 @@
      <!-- lifter -->
      <mimic joint="knee_joint"  offset="0.0" multiplier="-1.0"
-            P="4000" I="0.1" D="80" i_max="500" i_min="-500"
-            command_max="2000" command_min="-2000">
+            P="100" I="0.1" D="10" i_max="500" i_min="-500"
+            command_max="2000" command_min="-2000" velocity='true'>
        knee_joint_mimic
-       <joint> knee_joint </joint>
-       <offset> 0.0 </offset>
-       <multiplier> -1.0 </multiplier>
-       <P> 4000 </P>
-       <I> 0.1 </I>
-       <D> 80 </D>
-       <i_max>  500 </i_max>
-       <i_min> -500 </i_min>
-       <command_max>  2000 </command_max>
-       <command_min> -2000 </command_min>
      </mimic>
      <mimic joint="ankle_joint"  offset="0.0" multiplier="-1.0"
-            P="4000" I="0.1" D="80" i_max="500" i_min="-500"
-            command_max="2000" command_min="-2000">
+            P="100" I="0.1" D="10" i_max="500" i_min="-500"
+            command_max="2000" command_min="-2000" velocity='true'>
        ankle_joint_mimic
-       <joint> ankle_joint </joint>
-       <offset> 0.0 </offset>
-       <multiplier> -1.0 </multiplier>
-       <P> 4000 </P>
-       <I> 0.1 </I>
-       <D> 80 </D>
-       <i_max>  500 </i_max>
-       <i_min> -500 </i_min>
-       <command_max>  2000 </command_max>
-       <command_min> -2000 </command_min>
      </mimic>
      <!-- lifter(dummy) -->
      <mimic joint="knee_joint"  offset="0.0" multiplier="-1.0"
-            P="1000" I="0.0" D="1" i_max="0" i_min="0"
-            command_max="200" command_min="-200">
+            P="100" I="0.0" D="10" i_max="0" i_min="0"
+            command_max="200" command_min="-200" velocity='true'>
        knee_joint_dummy
-       <joint> knee_joint </joint>
-       <offset> 0.0 </offset>
-       <multiplier> -1.0 </multiplier>
-       <P> 1000 </P>
-       <I> 0.0 </I>
-       <D> 1 </D>
-       <i_max>  0 </i_max>
-       <i_min> -0 </i_min>
-       <command_max>  200 </command_max>
-       <command_min> -200 </command_min>
      </mimic>
      <mimic joint="ankle_joint"  offset="0.0" multiplier="1.0"
-            P="1000" I="0.0" D="1" i_max="0" i_min="0"
-            command_max="200" command_min="-200">
+            P="100" I="0.0" D="10" i_max="0" i_min="0"
+            command_max="200" command_min="-200"  velocity='true'>
        ankle_joint_dummy
-       <joint> ankle_joint </joint>
-       <offset> 0.0 </offset>
-       <multiplier> 1.0 </multiplier>
-       <P> 1000 </P>
-       <I> 0.0 </I>
-       <D> 1 </D>
-       <i_max>  0 </i_max>
-       <i_min> -0 </i_min>
-       <command_max>  200 </command_max>
-       <command_min> -200 </command_min>
      </mimic>
      <!-- lhand -->
@@ -102,14 +94,4 @@
             command_max="50" command_min="-50">
        l_indexbase_joint
-       <joint> l_thumb_joint </joint>
-       <offset> 0.0 </offset>
-       <multiplier> -1.0 </multiplier>
-       <P> 30 </P>
-       <I> 0.0 </I>
-       <D> 0.03 </D>
-       <i_max>  0 </i_max>
-       <i_min> -0 </i_min>
-       <command_max>  50 </command_max>
-       <command_min> -50 </command_min>
      </mimic>
      <mimic joint="l_thumb_joint"  offset="-0.2" multiplier="-0.3"
@@ -117,14 +99,4 @@
             command_max="50" command_min="-50">
        l_indexmid_joint
-       <joint> l_thumb_joint </joint>
-       <offset> -0.2 </offset>
-       <multiplier> -0.3 </multiplier>
-       <P> 30 </P>
-       <I> 0.0 </I>
-       <D> 0.03 </D>
-       <i_max>  0 </i_max>
-       <i_min> -0 </i_min>
-       <command_max>  50 </command_max>
-       <command_min> -50 </command_min>
      </mimic>
      <mimic joint="l_thumb_joint"  offset="-0.2" multiplier="-0.3"
@@ -132,14 +104,4 @@
             command_max="50" command_min="-50">
        l_indexend_joint
-       <joint> l_thumb_joint </joint>
-       <offset> -0.2 </offset>
-       <multiplier> -0.3 </multiplier>
-       <P> 30 </P>
-       <I> 0.0 </I>
-       <D> 0.03 </D>
-       <i_max>  0 </i_max>
-       <i_min> -0 </i_min>
-       <command_max>  50 </command_max>
-       <command_min> -50 </command_min>
      </mimic>
      <!-- rhand -->
@@ -148,14 +110,4 @@
             command_max="50" command_min="-50">
        r_indexbase_joint
-       <joint> r_thumb_joint </joint>
-       <offset> 0.0 </offset>
-       <multiplier> -1.0 </multiplier>
-       <P> 30 </P>
-       <I> 0.0 </I>
-       <D> 0.03 </D>
-       <i_max>  0 </i_max>
-       <i_min> -0 </i_min>
-       <command_max>  50 </command_max>
-       <command_min> -50 </command_min>
      </mimic>
      <mimic joint="r_thumb_joint"  offset="0.2" multiplier="-0.3"
@@ -163,14 +115,4 @@
             command_max="50" command_min="-50">
        r_indexmid_joint
-       <joint> r_thumb_joint </joint>
-       <offset> 0.2 </offset>
-       <multiplier> -0.3 </multiplier>
-       <P> 30 </P>
-       <I> 0.0 </I>
-       <D> 0.03 </D>
-       <i_max>  0 </i_max>
-       <i_min> -0 </i_min>
-       <command_max>  50 </command_max>
-       <command_min> -50 </command_min>
      </mimic>
      <mimic joint="r_thumb_joint"  offset="0.2" multiplier="-0.3"
@@ -178,14 +120,36 @@
             command_max="50" command_min="-50">
        r_indexend_joint
-       <joint> r_thumb_joint </joint>
-       <offset> 0.2 </offset>
-       <multiplier> -0.3 </multiplier>
-       <P> 30 </P>
-       <I> 0.0 </I>
-       <D> 0.03 </D>
-       <i_max>  0 </i_max>
-       <i_min> -0 </i_min>
-       <command_max>  50 </command_max>
-       <command_min> -50 </command_min>
+     </mimic>
+      <!-- r_elbow -->
+     <mimic joint="r_elbow_joint"  offset="0.0" multiplier="-1.0"
+            P="100" I="0.01" D="10" i_max="0" i_min="-0"
+            command_max="50" command_min="-50" velocity='true'>
+       r_elbow_joint_mimic
+     </mimic>
+     <mimic joint="r_elbow_joint"  offset="0.0" multiplier="0.591"
+            P="100" I="0.01" D="10" i_max="0" i_min="-0"
+            command_max="50" command_min="-50" velocity='true'>
+       r_elbow_middle_joint
+     </mimic>
+     <mimic joint="r_elbow_joint"  offset="0.0" multiplier="0.409"
+            P="100" I="0.01" D="10" i_max="0" i_min="-0"
+            command_max="50" command_min="-50" velocity='true'>
+       r_elbow_middle_joint_mimic
+     </mimic>
+     <!-- l_elbow -->
+     <mimic joint="l_elbow_joint"  offset="0.0" multiplier="-1.0"
+            P="100" I="0.01" D="10" i_max="0" i_min="-0"
+            command_max="50" command_min="-50" velocity='true'>
+       l_elbow_joint_mimic
+     </mimic>
+     <mimic joint="l_elbow_joint"  offset="0.0" multiplier="0.591"
+            P="100" I="0.01" D="10" i_max="0" i_min="-0"
+            command_max="50" command_min="-50" velocity='true'>
+       l_elbow_middle_joint
+     </mimic>
+     <mimic joint="l_elbow_joint"  offset="0.0" multiplier="0.409"
+            P="100" I="0.01" D="10" i_max="0" i_min="-0"
+            command_max="50" command_min="-50" velocity='true'>
+       l_elbow_middle_joint_mimic
      </mimic>
    </plugin>

File: seed_r7_description/urdf/typeF_upperbody/noid_upper_typef.urdf.xacro (robot description, xacro)
@@ -145,7 +145,43 @@
   </link>
   <xacro:gazebo_link_reference link_name="l_upperarm_link" />
+  <link name="l_elbow_virtual_link">
+    <inertial>
+      <mass value="0.001" />
+      <origin xyz="0 0 0" rpy="0 0 0"/>
+      <inertia ixx="0.01" ixy="0" ixz="0" iyy="0.01" iyz="0" izz="0.01"/>
+    </inertial>
+  </link>
+  <xacro:gazebo_link_reference link_name="l_elbow_virtual_link" />
+  <link name="l_elbow_virtual_link_dummy">
+    <inertial>
+      <mass value="0.001" />
+      <origin xyz="0 0 0" rpy="0 0 0"/>
+      <inertia ixx="0.01" ixy="0" ixz="0" iyy="0.01" iyz="0" izz="0.01"/>
+    </inertial>
+  </link>
+  <xacro:gazebo_link_reference link_name="l_elbow_virtual_link_dummy" />
+  <link name="l_elbow_middle_link">
+    <xacro:unless value="${disable_mesh}"> <visual>
+      <origin xyz="0 0 0" rpy="0 -0 0"/>
+      <geometry>
+        <mesh filename="package://seed_r7_description/meshes/typeF_upperbody/elbow_middle_link.dae" scale="1 1 1" />
+      </geometry>
+    </visual> </xacro:unless>
+    <xacro:unless value="${disable_mesh}"> <collision>
+      <origin xyz="0 0 0" rpy="0 -0 0"/>
+      <geometry>
+        <mesh filename="package://seed_r7_description/meshes/typeF_upperbody/elbow_middle_link.dae" scale="1 1 1" />
+      </geometry>
+    </collision> </xacro:unless>
+    <inertial>
+      <mass value="0.162" />
+      <origin xyz="-0.014 0 -0.032" rpy="0 -0 0"/>
+      <inertia ixx="0.00178" ixy="0" ixz="0" iyy="0.00179" iyz="0" izz="0.0035"/>
+    </inertial>
+  </link>
+  <xacro:gazebo_link_reference link_name="l_elbow_middle_link" />
   <link name="l_elbow_link">
     <xacro:unless value="${disable_mesh}"> <visual>
-      <origin xyz="-0.035 0 -0.035" rpy="0 -0 0"/>
+      <origin xyz="0 0 0" rpy="0 -0 0"/>
       <geometry>
         <mesh filename="package://seed_r7_description/meshes/typeF_upperbody/LARM_LINK4_mesh.dae" scale="1 1 1" />
@@ -153,5 +189,5 @@
     </visual> </xacro:unless>
     <xacro:unless value="${disable_mesh}"> <collision>
-      <origin xyz="-0.035 0 -0.035" rpy="0 -0 0"/>
+      <origin xyz="0 0 0" rpy="0 -0 0"/>
       <geometry>
         <mesh filename="package://seed_r7_description/meshes/typeF_upperbody/LARM_LINK4_mesh.dae" scale="1 1 1" />
@@ -324,7 +360,43 @@
   </link>
   <xacro:gazebo_link_reference link_name="r_upperarm_link" />
+  <link name="r_elbow_virtual_link">
+    <inertial>
+      <mass value="0.001" />
+      <origin xyz="0 0 0" rpy="0 0 0"/>
+      <inertia ixx="0.01" ixy="0" ixz="0" iyy="0.01" iyz="0" izz="0.01"/>
+    </inertial>
+  </link>
+  <xacro:gazebo_link_reference link_name="r_elbow_virtual_link" />
+  <link name="r_elbow_virtual_link_dummy">
+    <inertial>
+      <mass value="0.001" />
+      <origin xyz="0 0 0" rpy="0 0 0"/>
+      <inertia ixx="0.01" ixy="0" ixz="0" iyy="0.01" iyz="0" izz="0.01"/>
+    </inertial>
+  </link>
+  <xacro:gazebo_link_reference link_name="r_elbow_virtual_link_dummy" />
+  <link name="r_elbow_middle_link">
+    <xacro:unless value="${disable_mesh}"> <visual>
+      <origin xyz="0 0 0" rpy="0 -0 0"/>
+      <geometry>
+        <mesh filename="package://seed_r7_description/meshes/typeF_upperbody/elbow_middle_link.dae" scale="1 1 1" />
+      </geometry>
+    </visual> </xacro:unless>
+    <xacro:unless value="${disable_mesh}"> <collision>
+      <origin xyz="0 0 0" rpy="0 -0 0"/>
+      <geometry>
+        <mesh filename="package://seed_r7_description/meshes/typeF_upperbody/elbow_middle_link.dae" scale="1 1 1" />
+      </geometry>
+    </collision> </xacro:unless>
+    <inertial>
+      <mass value="0.162" />
+      <origin xyz="-0.014 0 -0.032" rpy="0 -0 0"/>
+      <inertia ixx="0.00178" ixy="0" ixz="0" iyy="0.00179" iyz="0" izz="0.0035"/>
+    </inertial>
+  </link>
+  <xacro:gazebo_link_reference link_name="r_elbow_middle_link" />
   <link name="r_elbow_link">
     <xacro:unless value="${disable_mesh}"> <visual>
-      <origin xyz="-0.035 0 -0.035" rpy="0 -0 0"/>
+      <origin xyz="0 0 0" rpy="0 -0 0"/>
       <geometry>
         <mesh filename="package://seed_r7_description/meshes/typeF_upperbody/RARM_LINK4_mesh.dae" scale="1 1 1" />
@@ -332,5 +404,5 @@
     </visual> </xacro:unless>
     <xacro:unless value="${disable_mesh}"> <collision>
-      <origin xyz="-0.035 0 -0.035" rpy="0 -0 0"/>
+      <origin xyz="0 0 0" rpy="0 -0 0"/>
       <geometry>
         <mesh filename="package://seed_r7_description/meshes/typeF_upperbody/RARM_LINK4_mesh.dae" scale="1 1 1" />
@@ -436,18 +508,8 @@
   </joint>
   <xacro:gazebo_transmission joint_name="l_shoulder_y_joint" />
-  <joint name="l_elbow_joint" type="revolute">
-    <parent link="l_upperarm_link"/>
-    <child  link="l_elbow_link"/>
-    <origin xyz="0.035 0 -0.1625" rpy="0 -0 0 "/>
-    <axis   xyz="0 1 0"/>
-    <!-- from -171 to 0 degrees-->
-    <limit lower="-3.0" upper="0" effort="100" velocity="1.2" />
-    <dynamics damping="0.2" friction="0" />
-  </joint>
-  <xacro:gazebo_transmission joint_name="l_elbow_joint" />
   <joint name="l_wrist_y_joint" type="revolute">
     <parent link="l_elbow_link"/>
     <child  link="l_forearm_link"/>
-    <origin xyz="-0.035 0 -0.070" rpy="0 -0 0 "/>
+    <origin xyz="0 0 -0.0355" rpy="0 -0 0 "/>
     <axis   xyz="0 0 1"/>
     <!-- from -180 to 180 degrees-->
@@ -536,18 +598,8 @@
   </joint>
   <xacro:gazebo_transmission joint_name="r_shoulder_y_joint" />
-  <joint name="r_elbow_joint" type="revolute">
-    <parent link="r_upperarm_link"/>
-    <child  link="r_elbow_link"/>
-    <origin xyz="0.035 0 -0.1625" rpy="0 -0 0 "/>
-    <axis   xyz="0 1 0"/>
-    <!-- from -171 to 0 degrees-->
-    <limit lower="-3.0" upper="0" effort="100" velocity="1.2" />
-    <dynamics damping="0.2" friction="0" />
-  </joint>
-  <xacro:gazebo_transmission joint_name="r_elbow_joint" />
   <joint name="r_wrist_y_joint" type="revolute">
     <parent link="r_elbow_link"/>
     <child  link="r_forearm_link"/>
-    <origin xyz="-0.035 0 -0.070" rpy="0 -0 0 "/>
+    <origin xyz="0 0 -0.0355" rpy="0 -0 0 "/>
     <axis   xyz="0 0 1"/>
     <!-- from -180 to 180 degrees-->
@@ -576,4 +628,79 @@
   </joint>
   <xacro:gazebo_transmission joint_name="r_wrist_r_joint" />
+  <joint name="r_elbow_joint" type="revolute">
+    <parent link="r_upperarm_link"/>
+    <child  link="r_elbow_virtual_link"/>
+    <origin xyz="0.0 0 -0.128" rpy="0 -0 0 "/>
+    <axis   xyz="0 1 0"/>
+    <!-- from -170 to 0 degrees-->
+    <limit lower="-3.0" upper="0" effort="100" velocity="1.1" />
+    <dynamics damping="0.2" friction="0.1" />
+  </joint>
+  <xacro:gazebo_transmission joint_name="r_elbow_joint" />
+  <joint name="r_elbow_joint_mimic" type="continuous">
+    <parent link="r_elbow_virtual_link"/>
+    <child  link="r_elbow_virtual_link_dummy"/>
+    <origin xyz="0.0 0 0" rpy="0 0 0 "/>
+    <axis   xyz="0 1 0"/>
+    <mimic joint="r_elbow_joint" multiplier="-1" offset="0" />
+  </joint>
+  <joint name="r_elbow_middle_joint" type="continuous">
+    <parent link="r_elbow_virtual_link_dummy"/>
+    <child  link="r_elbow_middle_link"/>
+    <origin xyz="0.0 0 0" rpy="0 -0 0 "/>
+    <axis   xyz="0 1 0"/>
+    <mimic joint="r_elbow_joint" multiplier="0.591222" offset="0" />
+  </joint>
+  <joint name="r_elbow_middle_joint_mimic" type="continuous">
+    <parent link="r_elbow_middle_link"/>
+    <child  link="r_elbow_link"/>
+    <origin xyz="0.0 0 -0.07" rpy="0 -0 0 "/>
+    <axis   xyz="0 1 0"/>
+    <mimic joint="r_elbow_joint" multiplier="0.408778" offset="0" />
+  </joint>
+  <joint name="l_elbow_joint" type="revolute">
+    <parent link="l_upperarm_link"/>
+    <child  link="l_elbow_virtual_link"/>
+    <origin xyz="0.0 0 -0.128" rpy="0 -0 0 "/>
+    <axis   xyz="0 1 0"/>
+    <!-- from -170 to 0 degrees-->
+    <limit lower="-3.0" upper="0" effort="100" velocity="1.1" />
+    <dynamics damping="0.2" friction="0.1" />
+  </joint>
+  <xacro:gazebo_transmission joint_name="l_elbow_joint" />
+  <joint name="l_elbow_joint_mimic" type="continuous">
+    <parent link="l_elbow_virtual_link"/>
+    <child  link="l_elbow_virtual_link_dummy"/>
+    <origin xyz="0.0 0 0" rpy="0 0 0 "/>
+    <axis   xyz="0 1 0"/>
+    <mimic joint="l_elbow_joint" multiplier="-1" offset="0" />
+  </joint>
+  <joint name="l_elbow_middle_joint" type="continuous">
+    <parent link="l_elbow_virtual_link_dummy"/>
+    <child  link="l_elbow_middle_link"/>
+    <origin xyz="0.0 0 0" rpy="0 -0 0 "/>
+    <axis   xyz="0 1 0"/>
+    <mimic joint="l_elbow_joint" multiplier="0.591222" offset="0" />
+  </joint>
+  <joint name="l_elbow_middle_joint_mimic" type="continuous">
+    <parent link="l_elbow_middle_link"/>
+    <child  link="l_elbow_link"/>
+    <origin xyz="0.0 0 -0.07" rpy="0 -0 0 "/>
+    <axis   xyz="0 1 0"/>
+    <mimic joint="l_elbow_joint" multiplier="0.408778" offset="0" />
+  </joint>
+    <!-- camera -->
+  <link name="chest_camera_link"/>
+  <joint name="body_link_to_chest_camera_link" type="fixed">
+    <parent  link="body_link"/>
+    <child link="chest_camera_link"/>
+    <origin xyz="0.062143 0.0 0.322289 " rpy="0 0.785398 0"/>
+  </joint>
+  <link name="chest_camera_right_ir_frame"/>
+  <joint name="chest_camera_link_to_chest_camera_right_ir_link" type="fixed">
+    <parent  link="chest_camera_link"/>
+    <child link="chest_camera_right_ir_frame"/>
+    <origin xyz="0 -0.055 0" rpy="0 0 0"/>  <!-- realsense d415-->
+  </joint>
   </xacro:macro>
 </robot>
