Commit message: base created new hand-urdf-model

File: seed_r7_description/urdf/trx_s/trx_s.urdf.xacro (robot description, xacro)
@@ -7,7 +7,7 @@
     <visual>
       <geometry>
-        <mesh filename="package://trx_s_ros_pkg/urdf/meshes/hand.DAE"/>
+        <mesh filename="package://seed_r7_description/meshes/trx_s/hand.DAE"/>
       </geometry>
-      <origin xyz="0 0 0" rpy="${M_PI} 0 ${reflect * M_PI / 2.0}"/>
+      <origin xyz="0 0 -0.031" rpy="${M_PI} 0 ${reflect * M_PI / 2.0}"/>
     </visual>
   </link>
@@ -15,8 +15,8 @@
   <link name="${prefix}_indexbase_link">
     <visual>
-      <geometry>"
-        <mesh filename="package://trx_s_ros_pkg/urdf/meshes/index_base.DAE"/>
+      <geometry>
+        <mesh filename="package://seed_r7_description/meshes/trx_s/index_base.DAE"/>
       </geometry>
-      <origin xyz="0 0 0" rpy="${M_PI} -0.57 ${reflect * M_PI / 2.0}"/>
+      <origin xyz="0 0 0" rpy="${M_PI} 0 ${reflect * M_PI / 2.0}"/>
     </visual>
   </link>
@@ -24,5 +24,5 @@
     <parent link="${prefix}_hand_link"/>
     <child  link="${prefix}_indexbase_link"/>
-    <origin xyz="0 0 -0.087" rpy="0 -0 0"/>
+    <origin xyz="0 ${-0.013*reflect} -0.087" rpy="0 0 0"/>
     <axis   xyz="1 0 0"/>
     <limit lower="-3.14159" upper="3.14159" effort="25" velocity="0.5" />
@@ -32,7 +32,7 @@
     <visual>
       <geometry>
-        <mesh filename="package://trx_s_ros_pkg/urdf/meshes/index_mid.DAE"/>
+        <mesh filename="package://seed_r7_description/meshes/trx_s/index_mid.DAE"/>
       </geometry>
-      <origin xyz="0 0 0" rpy="${M_PI} -0.57 ${reflect * M_PI / 2.0}"/>
+      <origin xyz="0 0 0" rpy="${M_PI} 0 ${reflect * M_PI / 2.0}"/>
     </visual>
   </link>
@@ -40,5 +40,5 @@
     <parent link="${prefix}_indexbase_link"/>
     <child  link="${prefix}_indexmid_link"/>
-    <origin xyz="0 0 -0.045" rpy="0 0.52 0 "/>
+    <origin xyz="0 0 -0.045" rpy="${0.52*reflect} 0 0 "/>
     <axis   xyz="1 0 0"/>
     <limit lower="-3.14159" upper="3.14159" effort="25" velocity="0.5" />
@@ -48,7 +48,7 @@
     <visual>
       <geometry>
-        <mesh filename="package://trx_s_ros_pkg/urdf/meshes/index_end.DAE"/>
+        <mesh filename="package://seed_r7_description/meshes/trx_s/index_end.DAE"/>
       </geometry>
-      <origin xyz="0 0 -0.025" rpy="0 0 0"/>
+      <origin xyz="0 0 0" rpy="${M_PI} 0 ${reflect * M_PI / 2.0}"/>
     </visual>
   </link>
@@ -56,5 +56,5 @@
     <parent link="${prefix}_indexmid_link"/>
     <child  link="${prefix}_indexend_link"/>
-    <origin xyz="-0.0 0 0.0" rpy="0 0 0 "/>
+    <origin xyz="0 ${-0.005*reflect} -0.025" rpy="${-1.13*reflect} 0 0 "/>
     <axis   xyz="1 0 0"/>
     <limit lower="-3.14159" upper="3.14159" effort="25" velocity="0.5" />
@@ -64,7 +64,7 @@
     <visual>
       <geometry>
-        <mesh filename="package://trx_s_ros_pkg/urdf/meshes/thumb.DAE"/>
+        <mesh filename="package://seed_r7_description/meshes/trx_s/thumb.DAE"/>
       </geometry>
-      <origin xyz="0 0 0" rpy="0 0 0 "/>
+      <origin xyz="0 0 0" rpy="${M_PI} 0 ${reflect * M_PI / 2.0}"/>
     </visual>
   </link>
@@ -72,7 +72,7 @@
     <parent  link="${prefix}_hand_link"/>
     <child  link="${prefix}_thumb_link"/>
-    <origin xyz="0.023 0 -0.054" rpy="${M_PI} 0+1 ${reflect * M_PI / 2.0}"/>
+    <origin xyz="0 ${0.023*reflect} -0.054" rpy="${-0.08 * reflect}  0 0"/>
     <axis   xyz="1 0 0"/>
-    <limit lower="-3.14159" upper="3.14159" effort="25" velocity="0.5" />
+    <limit lower="${-1.57 * (1 + reflect)/2.0}" upper="${1.57 * (1 - reflect)/2.0}" effort="25" velocity="0.5" />
   </joint>
   </xacro:macro>

File: seed_r7_description/urdf/typeF_upperbody/noid_upper_typef.urdf.xacro (robot description, xacro)
@@ -190,4 +190,10 @@
   <xacro:gazebo_link_reference link_name="l_forearm_link" />
   <link name="l_wrist_center">
+  <xacro:unless value="${disable_mesh}"> <visual>
+      <origin xyz="0 0 0" rpy="0 1.57 1.57"/>
+      <geometry>
+        <mesh filename="package://seed_r7_description/meshes/typeF_upperbody/wrist.dae" scale="1 1 1" />
+      </geometry>
+    </visual> </xacro:unless>
     <inertial>
       <mass value="0.05" />
@@ -369,4 +375,10 @@
   <xacro:gazebo_link_reference link_name="r_forearm_link" />
   <link name="r_wrist_center">
+   <xacro:unless value="${disable_mesh}"> <visual>
+      <origin xyz="0 0 0" rpy="0 1.57 1.57"/>
+      <geometry>
+        <mesh filename="package://seed_r7_description/meshes/typeF_upperbody/wrist.dae" scale="1 1 1" />
+      </geometry>
+    </visual> </xacro:unless>
     <inertial>
       <mass value="0.05" />

Commit message: hand stroke_converter changed

File: seed_r7_description/urdf/trx_s/trx_s.urdf.xacro (robot description, xacro)
@@ -56,7 +56,7 @@
     <parent link="${prefix}_hand_link"/>
     <child  link="${prefix}_indexbase_link"/>
-    <origin xyz="0 ${-0.013*reflect} -0.087" rpy="${reflect * -0.3} 0 0"/>
+    <origin xyz="0 ${-0.013*reflect} -0.087" rpy="${reflect * 0.75} 0 0"/>
     <axis   xyz="1 0 0"/>
-    <limit lower="-3.14159" upper="3.14159" effort="25" velocity="0.5" />
+    <limit lower="-0.87" upper="0.87" effort="25" velocity="0.5" />
   </joint>
 <!-- hand index middle -->
@@ -87,5 +87,5 @@
     <origin xyz="0 0 -0.045" rpy="${0.52*reflect} 0 0 "/>
     <axis   xyz="1 0 0"/>
-    <limit lower="-3.14159" upper="3.14159" effort="25" velocity="0.5" />
+    <limit lower="-0.87" upper="0.87" effort="25" velocity="0.5" />
   </joint>
 <!-- hand index end -->
@@ -116,5 +116,5 @@
     <origin xyz="0 ${-0.005*reflect} -0.025" rpy="${-1.13*reflect} 0 0 "/>
     <axis   xyz="1 0 0"/>
-    <limit lower="-3.14159" upper="3.14159" effort="25" velocity="0.5" />
+    <limit lower="-0.87" upper="0.87" effort="25" velocity="0.5" />
   </joint>
 <!-- hand finger -->
@@ -149,7 +149,7 @@
     <parent  link="${prefix}_hand_link"/>
     <child  link="${prefix}_thumb_link"/>
-    <origin xyz="0 ${0.023*reflect} -0.054" rpy="${-0.08 * reflect}  0 0"/>
+    <origin xyz="0 ${0.023*reflect} -0.054" rpy="${-0.75 * reflect}  0 0"/>
     <axis   xyz="1 0 0"/>
-    <limit lower="${-1.57 * (1 + reflect)/2.0}" upper="${1.57 * (1 - reflect)/2.0}" effort="25" velocity="0.5" />
+    <limit lower="-0.87" upper="0.87" effort="25" velocity="0.5" />
   </joint>
   <link name="${prefix}_eef_grasp_link"/>

Commit message: change index finger joint of trx from revloute to mimic

File: seed_r7_description/urdf/trx_s/trx_s.urdf.xacro (robot description, xacro)
@@ -124,34 +124,21 @@
   </link>
   <xacro:gazebo_link_reference link_name="${prefix}_thumb_link" />
-  <joint name="${prefix}_indexbase_joint" type="revolute">
+  <joint name="${prefix}_indexbase_joint" type="continuous">
     <parent link="${prefix}_hand_link"/>
     <child  link="${prefix}_indexbase_link"/>
     <origin xyz="0 ${-0.013 * reflect} -0.115" rpy="0 -0 0 "/>
     <axis   xyz="1 0 0"/>
-    <limit lower="-3.14159" upper="3.14159" effort="100" velocity="0.5" />
-    <dynamics damping="0.2" friction="0" />
+    <mimic joint="${prefix}_thumb_joint" multiplier="-1" offset="0"/>
   </joint>
-  <!--xacro:gazebo_joint_reference joint_name="${prefix}_indexbase_joint" /-->
-  <xacro:gazebo_transmission joint_name="${prefix}_indexbase_joint" />
-  <joint name="${prefix}_indexmid_joint" type="revolute">
+  <joint name="${prefix}_indexmid_joint" type="fixed">
     <parent link="${prefix}_indexbase_link"/>
     <child  link="${prefix}_indexmid_link"/>
     <origin xyz="0 ${0.028754 * reflect} -0.034615" rpy="0 -0 0 "/>
-    <axis   xyz="1 0 0"/>
-    <limit lower="-3.14159" upper="3.14159" effort="100" velocity="0.5" />
-    <dynamics damping="0.2" friction="0" />
   </joint>
-  <!--xacro:gazebo_joint_reference joint_name="${prefix}_indexmid_joint" /-->
-  <xacro:gazebo_transmission joint_name="${prefix}_indexmid_joint" />
-  <joint name="${prefix}_indexend_joint" type="revolute">
+  <joint name="${prefix}_indexend_joint" type="fixed">
     <parent link="${prefix}_indexmid_link"/>
     <child  link="${prefix}_indexend_link"/>
     <origin xyz="0 ${0.021716 * reflect} -0.013357" rpy="0 -0 0 "/>
-    <axis   xyz="1 0 0"/>
-    <limit lower="-3.14159" upper="3.14159" effort="100" velocity="0.5" />
-    <dynamics damping="0.2" friction="0" />
   </joint>
-  <!--xacro:gazebo_joint_reference joint_name="${prefix}_indexend_joint" /-->
-  <xacro:gazebo_transmission joint_name="${prefix}_indexend_joint" />
   <joint name="${prefix}_thumb_joint" type="revolute">
     <parent link="${prefix}_hand_link"/>
@@ -159,5 +146,5 @@
     <origin xyz="0 ${0.022355 * reflect} -0.079645" rpy="0 -0 0 "/>
     <axis   xyz="1 0 0"/>
-    <limit lower="-3.14159" upper="3.14159" effort="100" velocity="0.5" />
+    <limit lower="-1.0" upper="1.0" effort="50" velocity="0.5" />
     <dynamics damping="0.2" friction="0" />
   </joint>
