Commit message: corrected the range of motion of the wrist joint

File: seed_r7_description/urdf/typeG_arm/typeg_arm.urdf.xacro (robot description, xacro)
@@ -255,6 +255,6 @@
     <origin xyz="0.124 0 0" rpy="0 0 0 "/>
     <axis   xyz="0 0 1"/>
-    <!-- from -10 to 10 degrees-->
-    <limit lower="-0.17" upper="0.17" effort="100" velocity="1.05" />
+    <!-- from -7 to 7 degrees-->
+    <limit lower="-0.12" upper="0.12" effort="100" velocity="1.05" />
     <dynamics damping="0.2" friction="0" />
   </joint>
@@ -265,6 +265,6 @@
     <origin xyz="0 0 0" rpy="0 0 0 "/>
     <axis   xyz="0 1 0"/>
-    <!-- from -90 to 17 degrees-->
-    <limit lower="-0.30" upper="1.57" effort="100" velocity="1.4" />
+    <!-- from -20 to 90 degrees-->
+    <limit lower="-0.34" upper="1.57" effort="100" velocity="1.4" />
     <dynamics damping="0.2" friction="0" />
   </joint>
