Commit message: fix typeg_arm urdf and gazebo laubch & yaml

File: seed_r7_description/typeg_arm/arm.urdf.xacro (robot description, xacro)
@@ -9,3 +9,81 @@
  <xacro:arm-upper/>
  <xacro:noid-wheels base_link="base_link"/>
+<!-- gazebo settings -->
+ <!-- camera -->
+<xacro:property  name="camera_name" value="front_camera"/>
+<link name="${camera_name}_depth_optical_frame"/>
+<joint name="${camera_name}_depth_optical_joint" type="fixed">
+  <origin xyz="0 0 0" rpy="${-M_PI/2} 0 ${-M_PI/2}" />
+  <parent link="${camera_name}_link" />
+  <child link="${camera_name}_depth_optical_frame" />
+</joint>
+<xacro:gazebo_depth_camera link_name="${camera_name}_link"
+                      frame_name="${camera_name}_depth_optical_frame"
+                      camera_name="${camera_name}"/>
+<xacro:property  name="camera_name" value="rear_camera"/>
+<link name="${camera_name}_depth_optical_frame"/>
+<joint name="${camera_name}_depth_optical_joint" type="fixed">
+  <origin xyz="0 0 0" rpy="${-M_PI/2} 0 ${-M_PI/2}" />
+  <parent link="${camera_name}_link" />
+  <child link="${camera_name}_depth_optical_frame" />
+</joint>
+<xacro:gazebo_depth_camera link_name="${camera_name}_link"
+                      frame_name="${camera_name}_depth_optical_frame"
+                      camera_name="${camera_name}"/>
+ <!-- laser -->
+ <xacro:gazebo_laser_sensor link_name="wheels_base_laser_link"
+                            frame_name="wheels_base_laser_link" />
+ <!-- joint control -->
+ <xacro:gazebo_trajectory_controller />
+ <!-- mobile base -->
+ <xacro:gazebo_base_controller base_frame="base_link" />
+ <!-- mimic joints -->
+ <gazebo>
+   <plugin name="mimic_updater" filename="libmimic_plugin.so">
+     <!-- lifter -->
+     <mimic joint="knee_joint"  offset="0.0" multiplier="-1.0"
+            P="1000" I="0.01" D="1" i_max="0" i_min="0"
+            command_max="50" command_min="-50" velocity="true">
+       knee_joint_mimic
+     </mimic>
+     <mimic joint="ankle_joint"  offset="0.0" multiplier="-1.0"
+            P="1000" I="0.01" D="1" i_max="0" i_min="0"
+            command_max="50" command_min="-50" velocity="true">
+       ankle_joint_mimic
+     </mimic>
+     <!-- lifter(dummy) -->
+     <mimic joint="knee_joint"  offset="0.0" multiplier="-1.0"
+            P="100" I="0.01" D="1" i_max="0" i_min="0"
+            command_max="50" command_min="-50" velocity="true">
+       knee_joint_dummy
+     </mimic>
+     <mimic joint="ankle_joint"  offset="0.0" multiplier="1.0"
+            P="100" I="0.01" D="1" i_max="0" i_min="0"
+            command_max="50" command_min="-50"  velocity="true">
+       ankle_joint_dummy
+     </mimic>
+     <!-- hand -->
+     <mimic joint="r_thumb_joint"  offset="0.0" multiplier="-1.0"
+            P="10" I="0.0" D="1" i_max="0" i_min="0"
+            command_max="50" command_min="-50" velocity="true">
+       r_indexbase_joint
+     </mimic>
+    <!-- elbow -->
+     <mimic joint="elbow_joint"  offset="0.0" multiplier="-1.0"
+            P="50" I="0.01" D="1" i_max="0" i_min="-0"
+            command_max="50" command_min="-50" velocity="true">
+       elbow_joint_mimic
+     </mimic>
+     <mimic joint="elbow_joint"  offset="0.0" multiplier="0.591"
+            P="10" I="0.01" D="1" i_max="0" i_min="-0"
+            command_max="50" command_min="-50" velocity="true">
+       elbow_middle_joint
+     </mimic>
+     <mimic joint="elbow_joint"  offset="0.0" multiplier="0.409"
+            P="10" I="0.01" D="1" i_max="0" i_min="-0"
+            command_max="50" command_min="-50" velocity="true">
+       elbow_middle_joint_mimic
+     </mimic>
+   </plugin>
+ </gazebo>
 </robot>

File: seed_r7_description/urdf/typeG_arm/typeg_arm.urdf.xacro (robot description, xacro)
@@ -19,7 +19,7 @@
     </collision> </xacro:unless>
     <inertial>
-      <mass value="1.257" />
-      <origin xyz="0 0 0.0" rpy="0 0 0"/>
-      <inertia ixx="0.034" ixy="0" ixz="0" iyy="0.034" iyz="0" izz="0.018"/>
+      <mass value="0.820" />
+      <origin xyz="-0.001 0 0.005" rpy="0 0 0"/>
+      <inertia ixx="-0.00348" ixy="0" ixz="0" iyy="0.00199" iyz="0" izz="0.00545"/>
     </inertial>
   </link>
@@ -39,7 +39,7 @@
     </collision> </xacro:unless>
     <inertial>
-      <mass value="1.257" />
-      <origin xyz="0 0 0.0" rpy="0 -0 0"/>
-      <inertia ixx="0.034" ixy="0" ixz="0" iyy="0.034" iyz="0" izz="0.018"/>
+      <mass value="0.982" />
+      <origin xyz="-0.004 0 0.061" rpy="0 -0 0"/>
+      <inertia ixx="0.00186" ixy="0" ixz="0" iyy="0.00198" iyz="0" izz="0.00058"/>
     </inertial>
   </link>
@@ -59,7 +59,7 @@
     </collision> </xacro:unless>
     <inertial>
-     <mass value="0.574" />
-      <origin xyz="0.005 0 -0.0654" rpy="0 -0 0"/>
-      <inertia ixx="0.00214" ixy="0" ixz="0" iyy="0.00217" iyz="0" izz="0.003"/>
+     <mass value="0.496" />
+      <origin xyz="-0.012 0 0.142" rpy="0 -0 0"/>
+      <inertia ixx="0.00504" ixy="0" ixz="0" iyy="0.00516" iyz="0" izz="0.00074"/>
     </inertial>
   </link>
@@ -89,5 +89,5 @@
     </visual> </xacro:unless>
     <xacro:unless value="${disable_mesh}"> <collision>
-      <origin xyz="0 0 0" rpy="0 0.66008352 0"/>
+      <origin xyz="0 0 0" rpy="0 0.928689695 0"/>
       <geometry>
         <mesh filename="package://seed_r7_description/meshes/typeG_arm/elbow_middle_link.dae" scale="1 1 1" />
@@ -95,7 +95,7 @@
     </collision> </xacro:unless>
     <inertial>
-      <mass value="0.162" />
-      <origin xyz="-0.014 0 -0.032" rpy="0 -0 0"/>
-      <inertia ixx="0.00178" ixy="0" ixz="0" iyy="0.00179" iyz="0" izz="0.0035"/>
+      <mass value="0.193" />
+      <origin xyz="0.010 0 0.032" rpy="0 0.928689695 0"/>
+      <inertia ixx="0.00030" ixy="0" ixz="0" iyy="0.00030" iyz="0" izz="0.00011"/>
     </inertial>
   </link>
@@ -115,7 +115,7 @@
     </collision> </xacro:unless>
     <inertial>
-      <mass value="0.711" />
-      <origin xyz="-0.03 0 -0.0546" rpy="0 -0 0"/>
-      <inertia ixx="0.00178" ixy="0" ixz="0" iyy="0.00179" iyz="0" izz="0.0035"/>
+      <mass value="0.480" />
+      <origin xyz="0.069 0 0" rpy="0 -0 0"/>
+      <inertia ixx="0.00018" ixy="0" ixz="0" iyy="0.00045" iyz="0" izz="0.00047"/>
     </inertial>
   </link>
@@ -137,7 +137,7 @@
     </collision> </xacro:unless>
     <inertial>
-      <mass value="0.132" />
-      <origin xyz="0.006 0 -0.0738" rpy="0 -0 0"/>
-      <inertia ixx="0.0007" ixy="0" ixz="0" iyy="0.0007" iyz="0" izz="0.0004"/>
+      <mass value="0.262" />
+      <origin xyz="0.045 0 0" rpy="0 -0 0"/>
+      <inertia ixx="0.00020" ixy="0" ixz="0" iyy="0.00051" iyz="0" izz="0.00054"/>
     </inertial>
   </link>
@@ -157,7 +157,7 @@
     </collision> </xacro:unless>
     <inertial>
-      <mass value="0.05" />
+      <mass value="0.009" />
       <origin xyz="0 0 0" rpy="0 -0 0"/>
-      <inertia ixx="0.0001" ixy="0" ixz="0" iyy="0.0001" iyz="0" izz="0.0001"/>
+      <inertia ixx="0.00001" ixy="0" ixz="0" iyy="0.00001" iyz="0" izz="0.00001"/>
     </inertial>
   </link>
@@ -177,7 +177,7 @@
     </collision> </xacro:unless>
     <inertial>
-      <mass value="0.05" />
+      <mass value="0.025" />
       <origin xyz="0 0 0" rpy="0 -0 0"/>
-      <inertia ixx="0.0001" ixy="0" ixz="0" iyy="0.0001" iyz="0" izz="0.0001"/>
+      <inertia ixx="0.00001" ixy="0" ixz="0" iyy="0.00005" iyz="0" izz="0.00001"/>
     </inertial>
   </link>
@@ -276,5 +276,4 @@
     <!-- from -25 to 85 degrees-->
   </joint>
-  <xacro:gazebo_transmission joint_name="wrist_connector" />
   </xacro:macro>
 </robot>

Commit message: seed_r7_ros_pkg for cosmo

File: seed_r7_description/typeg_arm/arm.urdf.xacro (robot description, xacro)
@@ -9,81 +9,3 @@
  <xacro:arm-upper/>
  <xacro:noid-wheels base_link="base_link"/>
-<!-- gazebo settings -->
- <!-- camera -->
-<xacro:property  name="camera_name" value="front_camera"/>
-<link name="${camera_name}_depth_optical_frame"/>
-<joint name="${camera_name}_depth_optical_joint" type="fixed">
-  <origin xyz="0 0 0" rpy="${-M_PI/2} 0 ${-M_PI/2}" />
-  <parent link="${camera_name}_link" />
-  <child link="${camera_name}_depth_optical_frame" />
-</joint>
-<xacro:gazebo_depth_camera link_name="${camera_name}_link"
-                      frame_name="${camera_name}_depth_optical_frame"
-                      camera_name="${camera_name}"/>
-<xacro:property  name="camera_name" value="rear_camera"/>
-<link name="${camera_name}_depth_optical_frame"/>
-<joint name="${camera_name}_depth_optical_joint" type="fixed">
-  <origin xyz="0 0 0" rpy="${-M_PI/2} 0 ${-M_PI/2}" />
-  <parent link="${camera_name}_link" />
-  <child link="${camera_name}_depth_optical_frame" />
-</joint>
-<xacro:gazebo_depth_camera link_name="${camera_name}_link"
-                      frame_name="${camera_name}_depth_optical_frame"
-                      camera_name="${camera_name}"/>
- <!-- laser -->
- <xacro:gazebo_laser_sensor link_name="wheels_base_laser_link"
-                            frame_name="wheels_base_laser_link" />
- <!-- joint control -->
- <xacro:gazebo_trajectory_controller />
- <!-- mobile base -->
- <xacro:gazebo_base_controller base_frame="base_link" />
- <!-- mimic joints -->
- <gazebo>
-   <plugin name="mimic_updater" filename="libmimic_plugin.so">
-     <!-- lifter -->
-     <mimic joint="knee_joint"  offset="0.0" multiplier="-1.0"
-            P="1000" I="0.01" D="1" i_max="0" i_min="0"
-            command_max="50" command_min="-50" velocity="true">
-       knee_joint_mimic
-     </mimic>
-     <mimic joint="ankle_joint"  offset="0.0" multiplier="-1.0"
-            P="1000" I="0.01" D="1" i_max="0" i_min="0"
-            command_max="50" command_min="-50" velocity="true">
-       ankle_joint_mimic
-     </mimic>
-     <!-- lifter(dummy) -->
-     <mimic joint="knee_joint"  offset="0.0" multiplier="-1.0"
-            P="100" I="0.01" D="1" i_max="0" i_min="0"
-            command_max="50" command_min="-50" velocity="true">
-       knee_joint_dummy
-     </mimic>
-     <mimic joint="ankle_joint"  offset="0.0" multiplier="1.0"
-            P="100" I="0.01" D="1" i_max="0" i_min="0"
-            command_max="50" command_min="-50"  velocity="true">
-       ankle_joint_dummy
-     </mimic>
-     <!-- hand -->
-     <mimic joint="r_thumb_joint"  offset="0.0" multiplier="-1.0"
-            P="10" I="0.0" D="1" i_max="0" i_min="0"
-            command_max="50" command_min="-50" velocity="true">
-       r_indexbase_joint
-     </mimic>
-    <!-- elbow -->
-     <mimic joint="elbow_joint"  offset="0.0" multiplier="-1.0"
-            P="50" I="0.01" D="1" i_max="0" i_min="-0"
-            command_max="50" command_min="-50" velocity="true">
-       elbow_joint_mimic
-     </mimic>
-     <mimic joint="elbow_joint"  offset="0.0" multiplier="0.591"
-            P="10" I="0.01" D="1" i_max="0" i_min="-0"
-            command_max="50" command_min="-50" velocity="true">
-       elbow_middle_joint
-     </mimic>
-     <mimic joint="elbow_joint"  offset="0.0" multiplier="0.409"
-            P="10" I="0.01" D="1" i_max="0" i_min="-0"
-            command_max="50" command_min="-50" velocity="true">
-       elbow_middle_joint_mimic
-     </mimic>
-   </plugin>
- </gazebo>
 </robot>

File: seed_r7_description/urdf/typeG_arm/typeg_arm.urdf.xacro (robot description, xacro)
@@ -19,7 +19,7 @@
     </collision> </xacro:unless>
     <inertial>
-      <mass value="0.820" />
-      <origin xyz="-0.001 0 0.005" rpy="0 0 0"/>
-      <inertia ixx="-0.00348" ixy="0" ixz="0" iyy="0.00199" iyz="0" izz="0.00545"/>
+      <mass value="1.257" />
+      <origin xyz="0 0 0.0" rpy="0 0 0"/>
+      <inertia ixx="0.034" ixy="0" ixz="0" iyy="0.034" iyz="0" izz="0.018"/>
     </inertial>
   </link>
@@ -39,7 +39,7 @@
     </collision> </xacro:unless>
     <inertial>
-      <mass value="0.982" />
-      <origin xyz="-0.004 0 0.061" rpy="0 -0 0"/>
-      <inertia ixx="0.00186" ixy="0" ixz="0" iyy="0.00198" iyz="0" izz="0.00058"/>
+      <mass value="1.257" />
+      <origin xyz="0 0 0.0" rpy="0 -0 0"/>
+      <inertia ixx="0.034" ixy="0" ixz="0" iyy="0.034" iyz="0" izz="0.018"/>
     </inertial>
   </link>
@@ -59,7 +59,7 @@
     </collision> </xacro:unless>
     <inertial>
-     <mass value="0.496" />
-      <origin xyz="-0.012 0 0.142" rpy="0 -0 0"/>
-      <inertia ixx="0.00504" ixy="0" ixz="0" iyy="0.00516" iyz="0" izz="0.00074"/>
+     <mass value="0.574" />
+      <origin xyz="0.005 0 -0.0654" rpy="0 -0 0"/>
+      <inertia ixx="0.00214" ixy="0" ixz="0" iyy="0.00217" iyz="0" izz="0.003"/>
     </inertial>
   </link>
@@ -89,5 +89,5 @@
     </visual> </xacro:unless>
     <xacro:unless value="${disable_mesh}"> <collision>
-      <origin xyz="0 0 0" rpy="0 0.928689695 0"/>
+      <origin xyz="0 0 0" rpy="0 0.66008352 0"/>
       <geometry>
         <mesh filename="package://seed_r7_description/meshes/typeG_arm/elbow_middle_link.dae" scale="1 1 1" />
@@ -95,7 +95,7 @@
     </collision> </xacro:unless>
     <inertial>
-      <mass value="0.193" />
-      <origin xyz="0.010 0 0.032" rpy="0 0.928689695 0"/>
-      <inertia ixx="0.00030" ixy="0" ixz="0" iyy="0.00030" iyz="0" izz="0.00011"/>
+      <mass value="0.162" />
+      <origin xyz="-0.014 0 -0.032" rpy="0 -0 0"/>
+      <inertia ixx="0.00178" ixy="0" ixz="0" iyy="0.00179" iyz="0" izz="0.0035"/>
     </inertial>
   </link>
@@ -115,7 +115,7 @@
     </collision> </xacro:unless>
     <inertial>
-      <mass value="0.480" />
-      <origin xyz="0.069 0 0" rpy="0 -0 0"/>
-      <inertia ixx="0.00018" ixy="0" ixz="0" iyy="0.00045" iyz="0" izz="0.00047"/>
+      <mass value="0.711" />
+      <origin xyz="-0.03 0 -0.0546" rpy="0 -0 0"/>
+      <inertia ixx="0.00178" ixy="0" ixz="0" iyy="0.00179" iyz="0" izz="0.0035"/>
     </inertial>
   </link>
@@ -137,7 +137,7 @@
     </collision> </xacro:unless>
     <inertial>
-      <mass value="0.262" />
-      <origin xyz="0.045 0 0" rpy="0 -0 0"/>
-      <inertia ixx="0.00020" ixy="0" ixz="0" iyy="0.00051" iyz="0" izz="0.00054"/>
+      <mass value="0.132" />
+      <origin xyz="0.006 0 -0.0738" rpy="0 -0 0"/>
+      <inertia ixx="0.0007" ixy="0" ixz="0" iyy="0.0007" iyz="0" izz="0.0004"/>
     </inertial>
   </link>
@@ -157,7 +157,7 @@
     </collision> </xacro:unless>
     <inertial>
-      <mass value="0.009" />
+      <mass value="0.05" />
       <origin xyz="0 0 0" rpy="0 -0 0"/>
-      <inertia ixx="0.00001" ixy="0" ixz="0" iyy="0.00001" iyz="0" izz="0.00001"/>
+      <inertia ixx="0.0001" ixy="0" ixz="0" iyy="0.0001" iyz="0" izz="0.0001"/>
     </inertial>
   </link>
@@ -177,7 +177,7 @@
     </collision> </xacro:unless>
     <inertial>
-      <mass value="0.025" />
+      <mass value="0.05" />
       <origin xyz="0 0 0" rpy="0 -0 0"/>
-      <inertia ixx="0.00001" ixy="0" ixz="0" iyy="0.00005" iyz="0" izz="0.00001"/>
+      <inertia ixx="0.0001" ixy="0" ixz="0" iyy="0.0001" iyz="0" izz="0.0001"/>
     </inertial>
   </link>
@@ -276,4 +276,5 @@
     <!-- from -25 to 85 degrees-->
   </joint>
+  <xacro:gazebo_transmission joint_name="wrist_connector" />
   </xacro:macro>
 </robot>

File: seed_r7_description/urdf/typeG_lifter/lifter.urdf.xacro (robot description, xacro)
@@ -117,5 +117,5 @@
       <origin xyz="0 0 0.12" rpy="0 0 0"/>
       <axis xyz="0 -1 0"/>
-      <limit effort="200" lower="-1.5707" upper="0" velocity="0.5"/>
+      <limit effort="200" lower="-1.2" upper="0" velocity="0.5"/>
       <dynamics damping="0.2" friction="0" />
     </joint>
@@ -126,5 +126,5 @@
       <origin xyz="-0.012 0 0.035" rpy="0 0 0"/>
       <axis   xyz="0 -1 0"/>
-      <limit effort="200" lower="0" upper="1.5707" velocity="0.5" />
+      <limit effort="200" lower="0" upper="1.2" velocity="0.5" />
       <dynamics damping="0.2" friction="0" />
     </joint>
