Commit message: HA追加

File: seed_r7_description/ha/robot.urdf.xacro (robot description, xacro)
@@ -3,5 +3,5 @@
   <!-- The following included files set up definitions of parts of the robot body -->
   <!-- wraps upperbody and hand-->
-  <xacro:include filename="$(find seed_r7_description)/urdf/HA/ha.urdf.xacro" />
+  <xacro:include filename="$(find seed_r7_description)/urdf/HA/ha1.urdf.xacro" />
  <!-- Now we can start using the macros included above to define the actual robot -->
  <xacro:ha1 base_link="base_link"/>

File: seed_r7_description/urdf/HA/ha1.urdf.xacro (robot description, xacro)
@@ -47,4 +47,6 @@
     </inertial>
   </link>
+  <!-- eef link sample -->
+  <link name="ha_link"/>
   <joint name="ha1_1_joint" type="revolute">
     <parent link="${base_link}"/>
@@ -65,4 +67,13 @@
     <dynamics damping="0.2" friction="0" />
   </joint>
+  <joint name="ha_eef_joint" type="revolute">
+    <parent link="${base_link}"/>
+    <child  link="ha_link"/>
+    <origin xyz="0 -1 0" rpy="0 0 0 "/>
+    <axis   xyz="0 0 1"/>-->
+    <!-- from -180 to 180 degrees-->
+    <limit lower="-3.14" upper="3.14" effort="100" velocity="1.2" />
+    <dynamics damping="0.2" friction="0" />
+  </joint>
   </xacro:macro>
 </robot>
