Commit message: add rear laser

File: seed_r7_description/urdf/typeG_wheel/wheels.urdf.xacro (robot description, xacro)
@@ -150,4 +150,24 @@
     </link>
     <xacro:gazebo_link_reference link_name="wheels_base_laser_link" />
+    <link name="wheels_rear_laser_link">
+      <xacro:unless value="${disable_mesh}"> <visual>
+        <origin xyz="0.0 0.0 0.0" rpy="0 0 0"/>
+        <geometry>
+          <mesh filename="package://seed_r7_description/meshes/typeG_wheel/wheels_urg.dae" scale="1 1 1" />
+        </geometry>
+      </visual> </xacro:unless>
+      <xacro:unless value="${disable_mesh}"> <collision>
+        <origin xyz="0.0 0.0 -0.0124" rpy="0 -0 0"/>
+        <geometry>
+          <box size="0.08 0.1 0.07" />
+        </geometry>
+      </collision> </xacro:unless>
+      <inertial>
+        <mass value="0.2" />
+        <origin xyz="0 0 0" rpy="0 -0 0"/>
+        <inertia ixx="0.0528" ixy="0" ixz="0" iyy="0.0202" iyz="0" izz="0.0235"/>
+      </inertial>
+    </link>
+    <xacro:gazebo_link_reference link_name="wheels_rear_laser_link" />
     <joint name="base_link_to_wheel_base_link_connector" type="fixed">
       <parent link="${base_link}"/>
@@ -185,4 +205,9 @@
       <origin xyz="0.308 0 0.1014" rpy="0 0 0"/>
     </joint>
+    <joint name="wheels_body_to_rear_laser_connector" type="fixed">
+      <parent  link="wheel_base_link"/>
+      <child link="wheels_rear_laser_link"/>
+      <origin xyz="-0.308 0 0.1014" rpy="0 0 -3.141592"/>
+    </joint>
     <link name="front_camera_base_link"/>
     <joint name="wheel_base_link_to_front_camera_base_link" type="fixed">
@@ -195,5 +220,5 @@
       <parent  link="front_camera_base_link"/>
       <child link="front_camera_link"/>
-      <origin xyz="0 0.0175 0.0125" rpy="0 0 0"/>
+      <origin xyz="0 0.0325 0.0125" rpy="0 0 0"/>
     </joint>
     <link name="front_camera_right_ir_frame"/>
@@ -213,5 +238,5 @@
       <parent  link="rear_camera_base_link"/>
       <child link="rear_camera_link"/>
-      <origin xyz="0 0.0175 0.0125" rpy="0 0 0"/>
+      <origin xyz="0 0.0325 0.0125" rpy="0 0 0"/>
     </joint>
     <link name="rear_camera_right_ir_frame"/>
